File: keyboard-fullsize.kicad_pcb (KiCad board)
At the start: 2 copper layers, 210 parts, among them SW1 SW_Push, SW10 SW_Push, SW100 SW_Push, SW101 SW_Push, SW102 SW_Push, SW103 SW_Push, SW104 SW_Push, SW105 SW_Push, SW11 SW_Push, SW12 SW_Push, SW13 SW_Push, SW14 SW_Push, SW15 SW_Push, SW16 SW_Push, SW17 SW_Push, SW18 SW_Push, SW19 SW_Push, SW2 SW_Push, SW20 SW_Push, SW21 SW_Push, SW22 SW_Push, SW23 SW_Push, SW24 SW_Push, SW25 SW_Push, SW26 SW_Push, SW27 SW_Push, SW28 SW_Push, SW29 SW_Push, SW3 SW_Push, SW30 SW_Push, SW31 SW_Push, SW32 SW_Push, SW33 SW_Push, SW34 SW_Push, SW35 SW_Push, SW36 SW_Push, SW37 SW_Push, SW38 SW_Push, SW39 SW_Push, SW4 SW_Push, SW40 SW_Push, SW41 SW_Push, SW42 SW_Push, SW43 SW_Push, SW44 SW_Push, SW45 SW_Push, SW46 SW_Push, SW47 SW_Push, SW48 SW_Push, SW49 SW_Push, SW5 SW_Push, SW50 SW_Push, SW51 SW_Push, SW52 SW_Push, SW53 SW_Push, SW54 SW_Push, SW55 SW_Push, SW56 SW_Push, SW57 SW_Push, SW58 SW_Push, SW59 SW_Push, SW6 SW_Push, SW60 SW_Push, SW61 SW_Push, SW62 SW_Push, SW63 SW_Push, SW64 SW_Push, SW65 SW_Push, SW66 SW_Push, SW67 SW_Push, SW68 SW_Push, SW69 SW_Push, SW7 SW_Push, SW70 SW_Push, SW71 SW_Push, SW72 SW_Push, SW73 SW_Push, SW74 SW_Push, SW75 SW_Push, SW76 SW_Push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

Commit message: Footprints für alle Tastengrößen, README, Lizenz
- Projekt-fp-lib-table für MX_Only (Submodul MX_Alps_Hybrid)
- 17 Nicht-1u-Tasten auf passende Footprints getauscht, Schaltplan und PCB,
  Pads/Netze/Positionen unverändert
- README (EN/DE) mit Suche nach einem Gehäuse-Designer
- Lizenz CC BY-NC-SA 4.0
- CLAUDE.md mit Projektstand

Co-Authored-By: Claude Opus 5 (1M context) <noreply@anthropic.com>
Parts:
- SW100, SW75, SW93, SW94, SW95, SW97, SW98, SW99: footprint MX_Only:MXOnly-1U-NoLED -> MX_Only:MXOnly-1.25U-NoLED
- SW104, SW30: footprint MX_Only:MXOnly-1U-NoLED -> MX_Only:MXOnly-2U-NoLED
- SW38: footprint MX_Only:MXOnly-1U-NoLED -> MX_Only:MXOnly-1.5U-NoLED
- SW57, SW92: footprint MX_Only:MXOnly-1U-NoLED -> MX_Only:MXOnly-2U-VerticalStabilizers-NoLED
- SW58: footprint MX_Only:MXOnly-1U-NoLED -> MX_Only:MXOnly-1.75U-NoLED
- SW71: footprint MX_Only:MXOnly-1U-NoLED -> MX_Only:MXOnly-ISO-NoLED
- SW87: footprint MX_Only:MXOnly-1U-NoLED -> MX_Only:MXOnly-2.75U-NoLED
- SW96: footprint MX_Only:MXOnly-1U-NoLED -> MX_Only:MXOnly-6.25U-NoLED
