File: convertible-keyboard-pcb.kicad_pcb (KiCad board)
At the start: 2 copper layers, 210 parts, among them SW1 SW_Push, SW10 SW_Push, SW100 SW_Push, SW101 SW_Push, SW102 SW_Push, SW103 SW_Push, SW104 SW_Push, SW105 SW_Push, SW11 SW_Push, SW12 SW_Push, SW13 SW_Push, SW14 SW_Push, SW15 SW_Push, SW16 SW_Push, SW17 SW_Push, SW18 SW_Push, SW19 SW_Push, SW2 SW_Push, SW20 SW_Push, SW21 SW_Push, SW22 SW_Push, SW23 SW_Push, SW24 SW_Push, SW25 SW_Push, SW26 SW_Push, SW27 SW_Push, SW28 SW_Push, SW29 SW_Push, SW3 SW_Push, SW30 SW_Push, SW31 SW_Push, SW32 SW_Push, SW33 SW_Push, SW34 SW_Push, SW35 SW_Push, SW36 SW_Push, SW37 SW_Push, SW38 SW_Push, SW39 SW_Push, SW4 SW_Push, SW40 SW_Push, SW41 SW_Push, SW42 SW_Push, SW43 SW_Push, SW44 SW_Push, SW45 SW_Push, SW46 SW_Push, SW47 SW_Push, SW48 SW_Push, SW49 SW_Push, SW5 SW_Push, SW50 SW_Push, SW51 SW_Push, SW52 SW_Push, SW53 SW_Push, SW54 SW_Push, SW55 SW_Push, SW56 SW_Push, SW57 SW_Push, SW58 SW_Push, SW59 SW_Push, SW6 SW_Push, SW60 SW_Push, SW61 SW_Push, SW62 SW_Push, SW63 SW_Push, SW64 SW_Push, SW65 SW_Push, SW66 SW_Push, SW67 SW_Push, SW68 SW_Push, SW69 SW_Push, SW7 SW_Push, SW70 SW_Push, SW71 SW_Push, SW72 SW_Push, SW73 SW_Push, SW74 SW_Push, SW75 SW_Push, SW76 SW_Push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

Commit message: ANSI-Alternativen: Backslash, Enter und linkes Shift
- SW106 Backslash 1.5u (ROW2/COL13): ohne LED, Schalter auf der Platine um
  270° gedreht – nur so kollidiert er nicht mit dem ISO-Enter-Stabilisator
- SW107 Enter 2.25u (ROW3/COL13) und SW108 Shift links 2.25u (ROW4/COL0)
  auf denselben Matrixpositionen wie ISO-Enter bzw. ISO-Shift
- ISO-Enter SW71 im Schaltplan um 180° gedreht: Pin 2 = COL13, Pin 1 = Diode
- Footprints mit dem Schaltplan verknüpft (Pfade fehlten seit kbplacer)
- kbplacer-Leiterbahnen entfernt: sie laufen durch die LED-Pads der
  kommenden Beleuchtung, das Routing wird ohnehin neu gemacht

DRC: nur erwartete NPTH-Überlappungen zwischen ISO- und ANSI-Footprints
(Stabi-/Befestigungslöcher) und der noch fehlende Platinenumriss.

Co-Authored-By: Claude Opus 5 (1M context) <noreply@anthropic.com>
Parts:
- added D106: D, Diode_SMD:D_SOD-123, B.Cu at (290.8, 88.9)
- added D107: D, Diode_SMD:D_SOD-123, B.Cu at (299.5, 111.5)
- added D108: D, Diode_SMD:D_SOD-123, B.Cu at (55.1, 127.8)
- added SW106: SW_Push, MX_Only:MXOnly-1.5U-NoLED, F.Cu at (300.0, 85.7)
- added SW107: SW_Push, MX_Only:MXOnly-2.25U-NoLED, F.Cu at (292.9, 104.8)
- added SW108: SW_Push, MX_Only:MXOnly-2.25U-NoLED, F.Cu at (50.0, 123.8)
Connections:
- SW71 pad 1: COL13 -> Net-(D71-A)
- SW71 pad 2: Net-(D71-A) -> COL13
Routing:
- net ROW4: track 411.1 -> 0.00 mm
- net ROW1: track 409.6 -> 0.00 mm
- net ROW3: track 391.3 -> 0.00 mm
- net ROW5: track 388.1 -> 0.00 mm
- net ROW2: track 356.4 -> 0.00 mm
- net ROW0: track 328.6 -> 0.00 mm
- net COL12: track 139.0 -> 0.00 mm
- net COL11: track 137.0 -> 0.00 mm
- net COL10: track 137.0 -> 0.00 mm
- net COL3: track 127.5 -> 0.00 mm
- net COL1: track 123.5 -> 0.00 mm
- net COL9: track 116.9 -> 0.00 mm
- net COL0: track 109.7 -> 0.00 mm
- net COL16: track 104.8 -> 0.00 mm
- net COL15: track 104.8 -> 0.00 mm
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
Commit message: Einfarbige Hintergrundbeleuchtung (LEDs optional)
- Neues Symbol keyboard:SW_MX_LED: Einheit A Schalter (Pins wie
  SW_Push_45deg), Einheit B LED mit Pin 3 = Anode, Pin 4 = Kathode –
  passend zu den ai03-LED-Footprints (KiCads SW_Push_LED ist umgekehrt belegt)
- Alle Schalter außer ANSI-Backslash auf LED-Footprints umgestellt
- Blatt "Backlight": je Taste LED-Einheit + 1k-Vorwiderstand an +5V,
  Kathoden auf BL_K; AO3400A low-side als PWM-Treiber (BL_PWM)
- Caps-Lock- (SW58) und Num-Lock-LED (SW34) als Lock-Anzeige mit eigenem
  2N7002-Treiber (CAPS_LED, NUM_LED)
- LED-Kathode bei SW71, SW76, SW107 auf die andere Seite gelegt (FLIPPED),
  sonst zu nah an den Stabi-Löchern der ISO/ANSI-Alternativtaste;
  für ISO-Enter eigener Footprint lib/keyboard.pretty/MXOnly-ISO-FLIPPED
- Vorwiderstände auf B.Cu neben den Schaltern, bei den Alternativtasten
  in freie Bereiche verschoben

ERC meldet noch die unverbundenen Treiber-Eingänge und fehlende
Versorgungsquelle – beides kommt mit dem MCU-Blatt.

Co-Authored-By: Claude Opus 5 (1M context) <noreply@anthropic.com>
Parts:
- added Q1: AO3400A, Package_TO_SOT_SMD:SOT-23, F.Cu at (30.0, 175.0)
- added Q2: 2N7002, Package_TO_SOT_SMD:SOT-23, F.Cu at (40.0, 175.0)
- added Q3: 2N7002, Package_TO_SOT_SMD:SOT-23, F.Cu at (50.0, 175.0)
- added R1: 1k, Resistor_SMD:R_0603_1608Metric, B.Cu at (33.0, 42.1)
- added R10: 1k, Resistor_SMD:R_0603_1608Metric, B.Cu at (242.6, 42.1)
- added R100: 1k, Resistor_SMD:R_0603_1608Metric, B.Cu at (297.3, 146.9)
- added R101: 1k, Resistor_SMD:R_0603_1608Metric, B.Cu at (323.5, 146.9)
- added R102: 1k, Resistor_SMD:R_0603_1608Metric, B.Cu at (342.6, 146.9)
- added R103: 1k, Resistor_SMD:R_0603_1608Metric, B.Cu at (361.6, 146.9)
- added R104: 1k, Resistor_SMD:R_0603_1608Metric, B.Cu at (395.0, 146.9)
- added R105: 1k, Resistor_SMD:R_0603_1608Metric, B.Cu at (423.5, 146.9)
- added R107: 1k, Resistor_SMD:R_0603_1608Metric, B.Cu at (289.3, 112.0)
- added R108: 1k, Resistor_SMD:R_0603_1608Metric, B.Cu at (47.0, 133.5)
- added R11: 1k, Resistor_SMD:R_0603_1608Metric, B.Cu at (261.6, 42.1)
- added R12: 1k, Resistor_SMD:R_0603_1608Metric, B.Cu at (280.7, 42.1)
- added R121: 100, Resistor_SMD:R_0603_1608Metric, F.Cu at (60.0, 175.0)
- added R122: 100k, Resistor_SMD:R_0603_1608Metric, F.Cu at (70.0, 175.0)
- added R123: 100, Resistor_SMD:R_0603_1608Metric, F.Cu at (80.0, 175.0)
- added R124: 100k, Resistor_SMD:R_0603_1608Metric, F.Cu at (90.0, 175.0)
- added R125: 100, Resistor_SMD:R_0603_1608Metric, F.Cu at (100.0, 175.0)
- added R126: 100k, Resistor_SMD:R_0603_1608Metric, F.Cu at (110.0, 175.0)
- added R13: 1k, Resistor_SMD:R_0603_1608Metric, B.Cu at (299.7, 42.1)
- added R14: 1k, Resistor_SMD:R_0603_1608Metric, B.Cu at (323.5, 42.1)
- added R15: 1k, Resistor_SMD:R_0603_1608Metric, B.Cu at (342.6, 42.1)
- added R16: 1k, Resistor_SMD:R_0603_1608Metric, B.Cu at (361.6, 42.1)
- added R17: 1k, Resistor_SMD:R_0603_1608Metric, B.Cu at (33.0, 70.7)
- added R18: 1k, Resistor_SMD:R_0603_1608Metric, B.Cu at (52.1, 70.7)
- added R19: 1k, Resistor_SMD:R_0603_1608Metric, B.Cu at (71.1, 70.7)
- added R2: 1k, Resistor_SMD:R_0603_1608Metric, B.Cu at (71.1, 42.1)
- added R20: 1k, Resistor_SMD:R_0603_1608Metric, B.Cu at (90.2, 70.7)
- added R21: 1k, Resistor_SMD:R_0603_1608Metric, B.Cu at (109.2, 70.7)
- added R22: 1k, Resistor_SMD:R_0603_1608Metric, B.Cu at (128.3, 70.7)
- added R23: 1k, Resistor_SMD:R_0603_1608Metric, B.Cu at (147.3, 70.7)
- added R24: 1k, Resistor_SMD:R_0603_1608Metric, B.Cu at (166.4, 70.7)
- added R25: 1k, Resistor_SMD:R_0603_1608Metric, B.Cu at (185.4, 70.7)
- added R26: 1k, Resistor_SMD:R_0603_1608Metric, B.Cu at (204.5, 70.7)
- added R27: 1k, Resistor_SMD:R_0603_1608Metric, B.Cu at (223.5, 70.7)
- added R28: 1k, Resistor_SMD:R_0603_1608Metric, B.Cu at (242.6, 70.7)
- added R29: 1k, Resistor_SMD:R_0603_1608Metric, B.Cu at (261.6, 70.7)
- added R3: 1k, Resistor_SMD:R_0603_1608Metric, B.Cu at (90.2, 42.1)
- added R30: 1k, Resistor_SMD:R_0603_1608Metric, B.Cu at (290.2, 70.7)
- added R31: 1k, Resistor_SMD:R_0603_1608Metric, B.Cu at (323.5, 70.7)
- added R32: 1k, Resistor_SMD:R_0603_1608Metric, B.Cu at (342.6, 70.7)
- added R33: 1k, Resistor_SMD:R_0603_1608Metric, B.Cu at (361.6, 70.7)
- added R34: 1k, Resistor_SMD:R_0603_1608Metric, B.Cu at (385.4, 70.7)
- added R35: 1k, Resistor_SMD:R_0603_1608Metric, B.Cu at (404.5, 70.7)
- added R36: 1k, Resistor_SMD:R_0603_1608Metric, B.Cu at (423.5, 70.7)
- added R37: 1k, Resistor_SMD:R_0603_1608Metric, B.Cu at (442.6, 70.7)
- added R38: 1k, Resistor_SMD:R_0603_1608Metric, B.Cu at (37.8, 89.7)
- added R39: 1k, Resistor_SMD:R_0603_1608Metric, B.Cu at (61.6, 89.7)
- added R4: 1k, Resistor_SMD:R_0603_1608Metric, B.Cu at (109.2, 42.1)
- added R40: 1k, Resistor_SMD:R_0603_1608Metric, B.Cu at (80.6, 89.7)
- added R41: 1k, Resistor_SMD:R_0603_1608Metric, B.Cu at (99.7, 89.7)
- added R42: 1k, Resistor_SMD:R_0603_1608Metric, B.Cu at (118.7, 89.7)
- added R43: 1k, Resistor_SMD:R_0603_1608Metric, B.Cu at (137.8, 89.7)
- added R44: 1k, Resistor_SMD:R_0603_1608Metric, B.Cu at (156.8, 89.7)
- added R45: 1k, Resistor_SMD:R_0603_1608Metric, B.Cu at (175.9, 89.7)
- added R46: 1k, Resistor_SMD:R_0603_1608Metric, B.Cu at (194.9, 89.7)
- added R47: 1k, Resistor_SMD:R_0603_1608Metric, B.Cu at (214.0, 89.7)
- added R48: 1k, Resistor_SMD:R_0603_1608Metric, B.Cu at (233.0, 89.7)
- added R49: 1k, Resistor_SMD:R_0603_1608Metric, B.Cu at (252.1, 89.7)
- added R5: 1k, Resistor_SMD:R_0603_1608Metric, B.Cu at (128.3, 42.1)
- added R50: 1k, Resistor_SMD:R_0603_1608Metric, B.Cu at (271.1, 89.7)
- added R51: 1k, Resistor_SMD:R_0603_1608Metric, B.Cu at (323.5, 89.7)
- added R52: 1k, Resistor_SMD:R_0603_1608Metric, B.Cu at (342.6, 89.7)
- added R53: 1k, Resistor_SMD:R_0603_1608Metric, B.Cu at (361.6, 89.7)
- added R54: 1k, Resistor_SMD:R_0603_1608Metric, B.Cu at (385.4, 89.7)
- added R55: 1k, Resistor_SMD:R_0603_1608Metric, B.Cu at (404.5, 89.7)
- added R56: 1k, Resistor_SMD:R_0603_1608Metric, B.Cu at (423.5, 89.7)
- added R57: 1k, Resistor_SMD:R_0603_1608Metric, B.Cu at (442.6, 99.2)
- added R58: 1k, Resistor_SMD:R_0603_1608Metric, B.Cu at (40.2, 108.8)
- added R59: 1k, Resistor_SMD:R_0603_1608Metric, B.Cu at (66.4, 108.8)
- added R6: 1k, Resistor_SMD:R_0603_1608Metric, B.Cu at (156.8, 42.1)
- added R60: 1k, Resistor_SMD:R_0603_1608Metric, B.Cu at (85.4, 108.8)
- added R61: 1k, Resistor_SMD:R_0603_1608Metric, B.Cu at (104.5, 108.8)
- added R62: 1k, Resistor_SMD:R_0603_1608Metric, B.Cu at (123.5, 108.8)
- added R63: 1k, Resistor_SMD:R_0603_1608Metric, B.Cu at (142.6, 108.8)
- added R64: 1k, Resistor_SMD:R_0603_1608Metric, B.Cu at (161.6, 108.8)
- added R65: 1k, Resistor_SMD:R_0603_1608Metric, B.Cu at (180.7, 108.8)
- added R66: 1k, Resistor_SMD:R_0603_1608Metric, B.Cu at (199.7, 108.8)
- added R67: 1k, Resistor_SMD:R_0603_1608Metric, B.Cu at (218.8, 108.8)
- added R68: 1k, Resistor_SMD:R_0603_1608Metric, B.Cu at (237.8, 108.8)
- added R69: 1k, Resistor_SMD:R_0603_1608Metric, B.Cu at (256.9, 108.8)
- added R7: 1k, Resistor_SMD:R_0603_1608Metric, B.Cu at (175.9, 42.1)
- added R70: 1k, Resistor_SMD:R_0603_1608Metric, B.Cu at (275.9, 108.8)
- added R71: 1k, Resistor_SMD:R_0603_1608Metric, B.Cu at (297.3, 99.2)
- added R72: 1k, Resistor_SMD:R_0603_1608Metric, B.Cu at (385.4, 108.8)
- added R73: 1k, Resistor_SMD:R_0603_1608Metric, B.Cu at (404.5, 108.8)
- added R74: 1k, Resistor_SMD:R_0603_1608Metric, B.Cu at (423.5, 108.8)
- added R75: 1k, Resistor_SMD:R_0603_1608Metric, B.Cu at (35.4, 127.8)
- added R76: 1k, Resistor_SMD:R_0603_1608Metric, B.Cu at (56.8, 127.8)
- added R77: 1k, Resistor_SMD:R_0603_1608Metric, B.Cu at (75.9, 127.8)
- added R78: 1k, Resistor_SMD:R_0603_1608Metric, B.Cu at (94.9, 127.8)
- added R79: 1k, Resistor_SMD:R_0603_1608Metric, B.Cu at (114.0, 127.8)
- added R8: 1k, Resistor_SMD:R_0603_1608Metric, B.Cu at (194.9, 42.1)
- added R80: 1k, Resistor_SMD:R_0603_1608Metric, B.Cu at (133.0, 127.8)
- added R81: 1k, Resistor_SMD:R_0603_1608Metric, B.Cu at (152.1, 127.8)
- added R82: 1k, Resistor_SMD:R_0603_1608Metric, B.Cu at (171.1, 127.8)
- added R83: 1k, Resistor_SMD:R_0603_1608Metric, B.Cu at (190.2, 127.8)
- added R84: 1k, Resistor_SMD:R_0603_1608Metric, B.Cu at (209.2, 127.8)
- added R85: 1k, Resistor_SMD:R_0603_1608Metric, B.Cu at (228.3, 127.8)
- added R86: 1k, Resistor_SMD:R_0603_1608Metric, B.Cu at (247.3, 127.8)
- added R87: 1k, Resistor_SMD:R_0603_1608Metric, B.Cu at (283.1, 127.8)
- added R88: 1k, Resistor_SMD:R_0603_1608Metric, B.Cu at (342.6, 127.8)
- added R89: 1k, Resistor_SMD:R_0603_1608Metric, B.Cu at (385.4, 127.8)
- added R9: 1k, Resistor_SMD:R_0603_1608Metric, B.Cu at (214.0, 42.1)
- added R90: 1k, Resistor_SMD:R_0603_1608Metric, B.Cu at (404.5, 127.8)
- added R91: 1k, Resistor_SMD:R_0603_1608Metric, B.Cu at (423.5, 127.8)
- added R92: 1k, Resistor_SMD:R_0603_1608Metric, B.Cu at (442.6, 137.3)
- added R93: 1k, Resistor_SMD:R_0603_1608Metric, B.Cu at (35.4, 146.9)
- added R94: 1k, Resistor_SMD:R_0603_1608Metric, B.Cu at (59.2, 146.9)
- added R95: 1k, Resistor_SMD:R_0603_1608Metric, B.Cu at (83.0, 146.9)
- added R96: 1k, Resistor_SMD:R_0603_1608Metric, B.Cu at (154.5, 146.9)
- added R97: 1k, Resistor_SMD:R_0603_1608Metric, B.Cu at (225.9, 146.9)
- added R98: 1k, Resistor_SMD:R_0603_1608Metric, B.Cu at (249.7, 146.9)
- added R99: 1k, Resistor_SMD:R_0603_1608Metric, B.Cu at (273.5, 146.9)
- SW1, SW10, SW101, SW102, SW103, SW105, SW11, SW12, SW13, SW14, SW15, SW16, SW17, SW18, SW19, SW2, SW20, SW21, SW22, SW23, SW24, SW25, SW26, SW27, SW28, SW29, SW3, SW31, SW32, SW33, SW34, SW35, SW36, SW37, SW39, SW4, SW40, SW41, SW42, SW43, SW44, SW45, SW46, SW47, SW48, SW49, SW5, SW50, SW51, SW52, SW53, SW54, SW55, SW56, SW59, SW6, SW60, SW61, SW62, SW63, SW64, SW65, SW66, SW67, SW68, SW69, SW7, SW70, SW72, SW73, SW74, SW77, SW78, SW79, SW8, SW80, SW81, SW82, SW83, SW84, SW85, SW86, SW88, SW89, SW9, SW90, SW91: value SW_Push -> SW_MX_LED; footprint MX_Only:MXOnly-1U-NoLED -> MX_Only:MXOnly-1U
- SW100, SW75, SW93, SW94, SW95, SW97, SW98, SW99: value SW_Push -> SW_MX_LED; footprint MX_Only:MXOnly-1.25U-NoLED -> MX_Only:MXOnly-1.25U
- SW104, SW30: value SW_Push -> SW_MX_LED; footprint MX_Only:MXOnly-2U-NoLED -> MX_Only:MXOnly-2U
- SW107: value SW_Push -> SW_MX_LED; footprint MX_Only:MXOnly-2.25U-NoLED -> MX_Only:MXOnly-2.25U-FLIPPED
- SW108: value SW_Push -> SW_MX_LED; footprint MX_Only:MXOnly-2.25U-NoLED -> MX_Only:MXOnly-2.25U
- SW38: value SW_Push -> SW_MX_LED; footprint MX_Only:MXOnly-1.5U-NoLED -> MX_Only:MXOnly-1.5U
- SW57, SW92: value SW_Push -> SW_MX_LED; footprint MX_Only:MXOnly-2U-VerticalStabilizers-NoLED -> MX_Only:MXOnly-2U-VerticalStabilizers
- SW58: value SW_Push -> SW_MX_LED; footprint MX_Only:MXOnly-1.75U-NoLED -> MX_Only:MXOnly-1.75U
- SW71: value SW_Push -> SW_MX_LED; footprint MX_Only:MXOnly-ISO-NoLED -> keyboard:MXOnly-ISO-FLIPPED
- SW76: value SW_Push -> SW_MX_LED; footprint MX_Only:MXOnly-1U-NoLED -> MX_Only:MXOnly-1U-FLIPPED
- SW87: value SW_Push -> SW_MX_LED; footprint MX_Only:MXOnly-2.75U-NoLED -> MX_Only:MXOnly-2.75U
- SW96: value SW_Push -> SW_MX_LED; footprint MX_Only:MXOnly-6.25U-NoLED -> MX_Only:MXOnly-6.25U
- moved D108 5.91 mm to (53.5, 133.5), turned to 0 degrees
- moved D71 1.52 mm to (309.0, 99.2)

Commit message: MCU-Blatt: RP2040, USB-C, Stromversorgung; README und CLAUDE.md
- Blatt "MCU": RP2040 (QFN-56) mit W25Q16JVSS-Flash, 12-MHz-Quarz,
  AP2112K-3.3, USB-C (HRO TYPE-C-31-M-12, CC 5k1) mit USBLC6-2SC6,
  500-mA-Polyfuse, 27-Ω-Serienwiderständen, RESET- und BOOTSEL-Taster,
  SWD-Testpads, Entkopplung je Versorgungspin
- Alle 30 GPIOs belegt: GPIO0–20 COL0–20, GPIO21–26 ROW0–5,
  GPIO27 BL_PWM, GPIO28 CAPS_LED, GPIO29 NUM_LED
- Stabile UUIDs in den erzeugten Blättern, Beschriftungen aufgeräumt
- Neue Bauteile mit dem Schaltplan verknüpft, vorerst unplatziert unterhalb
  der Tasten

ERC: 0 Meldungen, Parität sauber. DRC: nur fehlender Umriss, die gewollten
ISO/ANSI-NPTH-Überlappungen und zwei Silkscreen-Hinweise.

Co-Authored-By: Claude Opus 5 (1M context) <noreply@anthropic.com>
Parts:
- added C201: 4n7, Capacitor_SMD:C_0603_1608Metric, F.Cu at (30.0, 175.0)
- added C202: 10u, Capacitor_SMD:C_0805_2012Metric, F.Cu at (40.0, 175.0)
- added C203: 10u, Capacitor_SMD:C_0805_2012Metric, F.Cu at (50.0, 175.0)
- added C204: 15p, Capacitor_SMD:C_0603_1608Metric, F.Cu at (60.0, 175.0)
- added C205: 15p, Capacitor_SMD:C_0603_1608Metric, F.Cu at (70.0, 175.0)
- added C206: 100n, Capacitor_SMD:C_0603_1608Metric, F.Cu at (80.0, 175.0)
- added C210: 100n, Capacitor_SMD:C_0603_1608Metric, F.Cu at (90.0, 175.0)
- added C211: 100n, Capacitor_SMD:C_0603_1608Metric, F.Cu at (100.0, 175.0)
- added C212: 100n, Capacitor_SMD:C_0603_1608Metric, F.Cu at (110.0, 175.0)
- added C213: 100n, Capacitor_SMD:C_0603_1608Metric, F.Cu at (120.0, 175.0)
- added C214: 100n, Capacitor_SMD:C_0603_1608Metric, F.Cu at (130.0, 175.0)
- added C215: 100n, Capacitor_SMD:C_0603_1608Metric, F.Cu at (140.0, 175.0)
- added C216: 100n, Capacitor_SMD:C_0603_1608Metric, F.Cu at (150.0, 175.0)
- added C217: 100n, Capacitor_SMD:C_0603_1608Metric, F.Cu at (160.0, 175.0)
- added C218: 1u, Capacitor_SMD:C_0603_1608Metric, F.Cu at (170.0, 175.0)
- added C219: 1u, Capacitor_SMD:C_0603_1608Metric, F.Cu at (180.0, 175.0)
- added C220: 100n, Capacitor_SMD:C_0603_1608Metric, F.Cu at (190.0, 175.0)
- added C221: 100n, Capacitor_SMD:C_0603_1608Metric, F.Cu at (200.0, 175.0)
- added F1: 500mA, Fuse:Fuse_1206_3216Metric, F.Cu at (210.0, 175.0)
- added J1: USB_C, Connector_USB:USB_C_Receptacle_HRO_TYPE-C-31-M-12, F.Cu at (220.0, 175.0)
- added R201: 5k1, Resistor_SMD:R_0603_1608Metric, F.Cu at (120.0, 185.0)
- added R202: 5k1, Resistor_SMD:R_0603_1608Metric, F.Cu at (130.0, 185.0)
- added R203: 1M, Resistor_SMD:R_0603_1608Metric, F.Cu at (140.0, 185.0)
- added R204: 27, Resistor_SMD:R_0603_1608Metric, F.Cu at (150.0, 185.0)
- added R205: 27, Resistor_SMD:R_0603_1608Metric, F.Cu at (160.0, 185.0)
- added R206: 1k, Resistor_SMD:R_0603_1608Metric, F.Cu at (170.0, 185.0)
- added R207: 1k, Resistor_SMD:R_0603_1608Metric, F.Cu at (180.0, 185.0)
- added R208: 10k, Resistor_SMD:R_0603_1608Metric, F.Cu at (190.0, 185.0)
- added SW201: SW_Push, Button_Switch_SMD:SW_SPST_TL3342, F.Cu at (200.0, 185.0)
- added SW202: SW_Push, Button_Switch_SMD:SW_SPST_TL3342, F.Cu at (210.0, 185.0)
- added TP1: SWCLK, TestPoint:TestPoint_Pad_D1.0mm, F.Cu at (220.0, 185.0)
- added TP2: SWDIO, TestPoint:TestPoint_Pad_D1.0mm, F.Cu at (30.0, 195.0)
- added TP3: RUN, TestPoint:TestPoint_Pad_D1.0mm, F.Cu at (40.0, 195.0)
- added TP4: GND, TestPoint:TestPoint_Pad_D1.0mm, F.Cu at (50.0, 195.0)
- added U1: RP2040, Package_DFN_QFN:QFN-56-1EP_7x7mm_P0.4mm_EP3.2x3.2mm, F.Cu at (60.0, 195.0)
- added U2: W25Q16JVSS, Package_SO:SOIC-8_5.3x5.3mm_P1.27mm, F.Cu at (70.0, 195.0)
- added U3: AP2112K-3.3, Package_TO_SOT_SMD:SOT-23-5, F.Cu at (80.0, 195.0)
- added U4: USBLC6-2SC6, Package_TO_SOT_SMD:SOT-23-6, F.Cu at (90.0, 195.0)
- added Y1: 12MHz, Crystal:Crystal_SMD_3225-4Pin_3.2x2.5mm, F.Cu at (100.0, 195.0)
- moved Q1 10.0 mm to (30.0, 185.0)
- moved Q2 10.0 mm to (40.0, 185.0)
- moved Q3 10.0 mm to (50.0, 185.0)
- moved R121 10.0 mm to (60.0, 185.0)
- moved R122 10.0 mm to (70.0, 185.0)
- moved R123 10.0 mm to (80.0, 185.0)
- moved R124 10.0 mm to (90.0, 185.0)
- moved R125 10.0 mm to (100.0, 185.0)
- moved R126 10.0 mm to (110.0, 185.0)
