File: convertible-keyboard-pcb.kicad_pcb (KiCad board)
At the start: 2 copper layers, 371 parts, among them J1 USB_C, Q1 AO3400A, Q2 2N7002, Q3 2N7002, SW1 SW_MX_LED, SW10 SW_MX_LED, SW100 SW_MX_LED, SW101 SW_MX_LED, SW102 SW_MX_LED, SW103 SW_MX_LED, SW104 SW_MX_LED, SW105 SW_MX_LED, SW106 SW_Push, SW107 SW_MX_LED, SW108 SW_MX_LED, SW11 SW_MX_LED, SW12 SW_MX_LED, SW13 SW_MX_LED, SW14 SW_MX_LED, SW15 SW_MX_LED, SW16 SW_MX_LED, SW17 SW_MX_LED, SW18 SW_MX_LED, SW19 SW_MX_LED, SW2 SW_MX_LED, SW20 SW_MX_LED, SW201 SW_Push, SW202 SW_Push, SW21 SW_MX_LED, SW22 SW_MX_LED, SW23 SW_MX_LED, SW24 SW_MX_LED, SW25 SW_MX_LED, SW26 SW_MX_LED, SW27 SW_MX_LED, SW28 SW_MX_LED, SW29 SW_MX_LED, SW3 SW_MX_LED, SW30 SW_MX_LED, SW31 SW_MX_LED, SW32 SW_MX_LED, SW33 SW_MX_LED, SW34 SW_MX_LED, SW35 SW_MX_LED, SW36 SW_MX_LED, SW37 SW_MX_LED, SW38 SW_MX_LED, SW39 SW_MX_LED, SW4 SW_MX_LED, SW40 SW_MX_LED, SW41 SW_MX_LED, SW42 SW_MX_LED, SW43 SW_MX_LED, SW44 SW_MX_LED, SW45 SW_MX_LED, SW46 SW_MX_LED, SW47 SW_MX_LED, SW48 SW_MX_LED, SW49 SW_MX_LED, SW5 SW_MX_LED, SW50 SW_MX_LED, SW51 SW_MX_LED, SW52 SW_MX_LED, SW53 SW_MX_LED, SW54 SW_MX_LED, SW55 SW_MX_LED, SW56 SW_MX_LED, SW57 SW_MX_LED, SW58 SW_MX_LED, SW59 SW_MX_LED, SW6 SW_MX_LED, SW60 SW_MX_LED, SW61 SW_MX_LED, SW62 SW_MX_LED, SW63 SW_MX_LED, SW64 SW_MX_LED, SW65 SW_MX_LED, SW66 SW_MX_LED, SW67 SW_MX_LED, SW68 SW_MX_LED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

Commit message: Eigene Caps-/Num-Lock-Anzeige über dem Navigationsblock
- Caps- und Num-Taste gehören wieder zur normalen Beleuchtung (BL_K) –
  bei eingeschaltetem Licht war der Lock-Zustand in der Taste kaum erkennbar
- Je Anzeige 1k an +5V und zwei LEDs parallel zur Wahl: 3 mm THT
  (D121 Caps, D123 Num) oder 0805 SMD (D122, D124), Treiber Q2/Q3 wie bisher
- Platz im Spalt zwischen Druck/Rollen/Pause und Einfg/Pos1/BildAuf, also auf
  dem TKL-Teil: bleibt auch nach dem Abbrechen des Ziffernblocks erhalten
- tools/sync_pcb.py: feste Positionen über "absolute" in place_override.json
- README (EN/DE) und CLAUDE.md angepasst

ERC 0, Parität sauber.

Co-Authored-By: Claude Opus 5 (1M context) <noreply@anthropic.com>
Parts:
- added D121: 3mm, LED_THT:LED_D3.0mm, F.Cu at (355.9, 51.0)
- added D122: 0805, LED_SMD:LED_0805_2012Metric, F.Cu at (357.2, 56.5)
- added D123: 3mm, LED_THT:LED_D3.0mm, F.Cu at (336.9, 51.0)
- added D124: 0805, LED_SMD:LED_0805_2012Metric, F.Cu at (338.1, 56.5)
- added R127: 1k, Resistor_SMD:R_0603_1608Metric, B.Cu at (362.0, 51.0)
- added R128: 1k, Resistor_SMD:R_0603_1608Metric, B.Cu at (343.0, 51.0)
Connections:
- SW34 pad 4: /Backlight/NUM_K -> /Backlight/BL_K
- SW58 pad 4: /Backlight/CAPS_K -> /Backlight/BL_K

Commit message: Lock-Anzeigen zusätzlich klassisch über dem Numpad (Standard)
- Zweites Paar Caps-/Num-Lock-Anzeigen rechts oben über dem Numpad:
  0805 bestückt (D126 Caps, D128 Num), 3-mm-THT vorgesehen (D125, D127, DNP)
- Paar über dem Navigationsblock bleibt für die TKL vorgesehen, alle LEDs DNP
- Jede Position mit eigenem 1k (R127–R130, bestückt), damit auch beide Paare
  gleichzeitig mit voller Helligkeit gehen; Treiber Q2/Q3 unverändert
- DNP wird in tools/sync_pcb.py auf die Footprints übertragen
- Generator: UUIDs zählen pro Blatt, Blatt-UUIDs hängen am Dateinamen –
  Ergänzungen auf einem Blatt verschieben die anderen nicht mehr
  (einmalige UUID-Änderung in allen erzeugten Blättern)
- README (EN/DE): beide Positionen, Wahl liegt beim Gehäuse-Designer

ERC 0, Parität sauber, DRC ohne neue Fehler.

Co-Authored-By: Claude Opus 5 (1M context) <noreply@anthropic.com>
Parts:
- added D125: 3mm, LED_THT:LED_D3.0mm, F.Cu at (427.4, 36.0)
- added D126: 0805, LED_SMD:LED_0805_2012Metric, F.Cu at (428.6, 41.5)
- added D127: 3mm, LED_THT:LED_D3.0mm, F.Cu at (408.3, 36.0)
- added D128: 0805, LED_SMD:LED_0805_2012Metric, F.Cu at (409.6, 41.5)
- added R129: 1k, Resistor_SMD:R_0603_1608Metric, B.Cu at (433.4, 36.0)
- added R130: 1k, Resistor_SMD:R_0603_1608Metric, B.Cu at (414.4, 36.0)
