File: convertible-keyboard-pcb.kicad_pcb (KiCad board)
At the start: 2 copper layers, 2.2 x 1.9 mm, 486 parts, among them J1 USB_C, J2 Pico-EZmate 78171-0004, J3 JST-SH SM04B-SRSS-TB, Q1 AO3400A, Q2 2N7002, Q3 2N7002, SW1 SW_Push, SW10 SW_Push, SW100 SW_Push, SW101 SW_Push, SW102 SW_Push, SW103 SW_Push, SW104 SW_Push, SW105 SW_Push, SW106 SW_Push, SW107 SW_Push, SW108 SW_Push, SW11 SW_Push, SW12 SW_Push, SW13 SW_Push, SW14 SW_Push, SW15 SW_Push, SW16 SW_Push, SW17 SW_Push, SW18 SW_Push, SW19 SW_Push, SW2 SW_Push, SW20 SW_Push, SW201 SW_Push, SW202 SW_Push, SW21 SW_Push, SW22 SW_Push, SW23 SW_Push, SW24 SW_Push, SW25 SW_Push, SW26 SW_Push, SW27 SW_Push, SW28 SW_Push, SW29 SW_Push, SW3 SW_Push, SW30 SW_Push, SW31 SW_Push, SW32 SW_Push, SW33 SW_Push, SW34 SW_Push, SW35 SW_Push, SW36 SW_Push, SW37 SW_Push, SW38 SW_Push, SW39 SW_Push, SW4 SW_Push, SW40 SW_Push, SW41 SW_Push, SW42 SW_Push, SW43 SW_Push, SW44 SW_Push, SW45 SW_Push, SW46 SW_Push, SW47 SW_Push, SW48 SW_Push, SW49 SW_Push, SW5 SW_Push, SW50 SW_Push, SW51 SW_Push, SW52 SW_Push, SW53 SW_Push, SW54 SW_Push, SW55 SW_Push, SW56 SW_Push, SW57 SW_Push, SW58 SW_Push, SW59 SW_Push, SW6 SW_Push, SW60 SW_Push, SW61 SW_Push, SW62 SW_Push, SW63 SW_Push, SW64 SW_Push, SW65 SW_Push, SW66 SW_Push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

Commit message: Platinenumriss und Sollbruchstelle, Alternativ-LEDs in der Stückliste
- Umriss: Tastenfeld + 1,3 mm rundum (Ecken r = 1 mm). Die 1,3 mm sind
  nötig, weil die Stabi-Löcher von Leertaste, Num 0 und Num+ über das reine
  Tastenfeld hinausragen. USB-C J1 sitzt bündig mit der Oberkante
- Sollbruchstelle: 2 mm breiter Schlitz bei x = 378,6 mit vier
  Mouse-Bite-Stegen (Footprint Breakaway_Tab_MouseBite, BRK1–BRK4). Jeder
  Steg hat einen lochfreien Kanal für bis zu drei Bahnen pro Lage:
  BRK1 COL17–COL20/CAPS_K/NUM_K, BRK2 ROW1/ROW2/+5V,
  BRK3 ROW3/ROW4/BL_K, BRK4 ROW5
- Tasten-LEDs mit Stücklistenfeldern Manufacturer, MPN und
  LCSC Alternatives (geprüft: C401114 MEIHUA MHT151WDT,
  C2827252 TUOZHAN P2-1206WYCS2-0.9T-F); Standard bleibt XL-3216UWC-FB.
  tools/led_variant.py pflegt die Felder mit
- README (EN/DE) und CLAUDE.md aktualisiert

ERC 0, Parität sauber, DRC ohne Fehler.

Co-Authored-By: Claude Opus 5 (1M context) <noreply@anthropic.com>
Parts:
- added BRK1: Breakaway_Tab, Breakaway_Tab_MouseBite, F.Cu at (378.6, 52.4)
- added BRK2: Breakaway_Tab, Breakaway_Tab_MouseBite, F.Cu at (378.6, 76.2)
- added BRK3: Breakaway_Tab, Breakaway_Tab_MouseBite, F.Cu at (378.6, 114.3)
- added BRK4: Breakaway_Tab, Breakaway_Tab_MouseBite, F.Cu at (378.6, 142.9)
- moved J1 1.93 mm to (57.1, 31.0)
Other:
- board size 2.2 x 1.9 mm -> 431.2 x 126.4 mm

Commit message: Tastenfeld geroutet
- Spalten vorn (Schalter zu Schalter), Zeilen hinten als Schiene unter jeder
  Tastenreihe, ROW1–ROW5 über die Kanäle der Mouse-Bite-Stege zum Numpad
- LED-Versorgung: +5V und BL_K als Schienen je Reihe, verbunden über
  Längsstränge am linken Rand und links neben dem Numpad, je ein Übergang
  über BRK2 (+5V) und BRK3 (BL_K)
- Kurze Verbindungen je Taste (Schalter → Diode, Widerstand → LED) als
  gleiche Vorlage
- Netzklassen: Default 0,2/0,15 mm, Power 0,4 mm (+5V, VBUS, BL_K),
  USB 0,25 mm; R204/R205 gedreht (Buchsenseite zum ESD-Schutz)
- 4100 Bahnen, rund 700 Durchkontaktierungen, erzeugt mit einem eigenen
  Rasterrouter (A*, echte Konturen und Designregeln)

DRC ohne Fehler. Offen: Verbindungen zum Controller und der Controller-
Bereich selbst.

Co-Authored-By: Claude Opus 5 (1M context) <noreply@anthropic.com>
Claude-Session: https://claude.ai/code/session_019Bb524k282LjrfvEdpjuYy
Parts:
- turned R204 to -90 degrees
- turned R205 to -90 degrees
Routing:
- net +5V: track 0.00 -> 2990.9 mm, vias 0 -> 344
- net /Backlight/BL_K: track 0.00 -> 2895.9 mm, vias 0 -> 351
- net ROW4: track 0.00 -> 459.5 mm
- net ROW2: track 0.00 -> 455.3 mm
- net ROW1: track 0.00 -> 435.8 mm
- net ROW3: track 0.00 -> 430.2 mm, vias 0 -> 2
- net ROW5: track 0.00 -> 407.6 mm
- net ROW0: track 0.00 -> 344.4 mm, vias 0 -> 2
- net COL12: track 0.00 -> 138.4 mm
- net COL10: track 0.00 -> 136.6 mm
- net COL11: track 0.00 -> 136.4 mm
- net COL6: track 0.00 -> 127.3 mm
- net COL3: track 0.00 -> 127.1 mm
- net COL0: track 0.00 -> 123.3 mm
- net COL1: track 0.00 -> 123.1 mm
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
Commit message: Controller-Bereich geroutet, GND-Flächen, Pintausch GPIO6/21-29
Controller-Block sitzt jetzt in der F4/F5-Lücke: USB-C mit ESD oben an der
Kante, RP2040 mit Flash, Quarz, Versorgung und Treibern im Streifen unter der
F-Reihe. Alle SMD-Bauteile auf B.Cu, also einseitige Bestückung; die vier
SWD-Testpads sind reines Kupfer auf F.Cu.

J2 (Pico-EZmate) und J3 (JST-SH) liegen im Footprint von J1 auf denselben
Netzen - es wird immer nur eine der drei Buchsen bestückt. Ihre Courtyards
entfallen auf der Platine, sonst meldet DRC eine Überlappung.

Routing in festen Kanälen (0,2 mm Bahnen im 0,35-mm-Raster): Spaltenleitungen
enden je mit einem Via auf der vorhandenen Leitung der Tastenspalte, die
Numpad-Leitungen queren den Steg BRK1 auf beiden Lagen kreuzungsfrei. GND als
Fläche auf F.Cu und B.Cu über dem TKL-Teil, mit vollem Pad-Anschluss und rund
100 Vias; über die Sollbruchstege läuft bewusst kein Kupfer.

Pintausch am RP2040 (in CLAUDE.md ausdrücklich erlaubt, QMK übernimmt die
Zuordnung): GPIO6 wird ROW0, GPIO21-23 die LED-Steuerung, GPIO24 COL6,
GPIO25-29 ROW1-ROW5. Damit verlassen Zeilen, Spalten und LED-Steuerung den
Chip jeweils in die Richtung, in die sie ohnehin müssen.

ERC 0, DRC ohne Meldung, Schaltplan-Parität 0.
Offen bleibt eine Verbindung: ROW5 von U1 Pin 41 (145,80/57,94) zu D96 Pad 1
(164,62/148,53). Die ziehe ich nicht weiter automatisch, sie wird in KiCad von
Hand gezogen; ein Via bei (144,9/59,2) und ein freies F.Cu-Band bis x 151,9
liegen als Vorarbeit bereit.

Co-Authored-By: Claude Opus 5 (1M context) <noreply@anthropic.com>
Claude-Session: https://claude.ai/code/session_019Bb524k282LjrfvEdpjuYy
Parts:
- TP1, TP2, TP3, TP4: moved to F.Cu
- moved U3 128.6 mm to (183.0, 54.3)
- moved C203 126.4 mm to (186.8, 54.3), turned to 90 degrees
- moved F1 107.0 mm to (154.6, 32.4)
- moved C202 106.8 mm to (154.6, 38.3)
- moved J2 99.5 mm to (147.6, 31.0)
- moved C201 93.1 mm to (140.9, 34.1)
- moved R203 93.1 mm to (140.9, 30.6)
- moved U4 90.5 mm to (147.6, 39.3)
- moved J1 90.5 mm to (147.6, 31.0)
- moved R202 89.6 mm to (151.6, 39.3)
- moved R204 88.9 mm to (144.3, 41.0)
- moved R201 88.6 mm to (140.9, 37.6)
- moved J3 88.0 mm to (147.6, 30.6)
- moved R205 83.7 mm to (142.6, 40.0)
- moved C210 82.7 mm to (166.8, 54.3), turned to 90 degrees
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Connections:
- U1 pad 32: ROW0 -> BL_PWM
- U1 pad 34: ROW1 -> CAPS_LED
- U1 pad 35: ROW2 -> NUM_LED
- U1 pad 36: ROW3 -> COL6
- U1 pad 37: ROW4 -> ROW1
- U1 pad 38: ROW5 -> ROW2
- U1 pad 39: BL_PWM -> ROW3
- U1 pad 40: CAPS_LED -> ROW4
- U1 pad 41: NUM_LED -> ROW5
- U1 pad 8: COL6 -> ROW0
Routing:
- net COL20: track 66.7 -> 383.0 mm
- net COL19: track 76.3 -> 369.9 mm, vias 0 -> 1
- net COL18: track 57.2 -> 329.6 mm, vias 0 -> 1
- net /Backlight/CAPS_K: track 0.00 -> 256.3 mm, vias 0 -> 2
- net COL17: track 80.0 -> 329.3 mm, vias 0 -> 1
- net /Backlight/NUM_K: track 0.00 -> 243.9 mm, vias 0 -> 1
- net COL16: track 104.8 -> 318.3 mm, vias 0 -> 1
- net COL15: track 104.9 -> 299.9 mm, vias 0 -> 1
- net COL14: track 104.8 -> 280.8 mm, vias 0 -> 1
- net COL13: track 95.1 -> 252.0 mm, vias 0 -> 1
- net +3V3: track 0.00 -> 153.1 mm, vias 0 -> 13
- net COL12: track 138.4 -> 275.7 mm, vias 0 -> 1
- net COL0: track 123.3 -> 247.2 mm, vias 0 -> 1
- net COL11: track 136.4 -> 255.4 mm, vias 0 -> 1
- net +5V: track 2990.9 -> 3099.4 mm, vias 344 -> 348
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- added copper zone on B.Cu, net GND
- added copper zone on F.Cu, net GND
