File: convertible-keyboard-pcb.kicad_sch (KiCad schematic)
At the start: 210 parts, among them SW1 SW_Push, SW10 SW_Push, SW100 SW_Push, SW101 SW_Push, SW102 SW_Push, SW103 SW_Push, SW104 SW_Push, SW105 SW_Push, SW11 SW_Push, SW12 SW_Push, SW13 SW_Push, SW14 SW_Push, SW15 SW_Push, SW16 SW_Push, SW17 SW_Push, SW18 SW_Push, SW19 SW_Push, SW2 SW_Push, SW20 SW_Push, SW21 SW_Push, SW22 SW_Push, SW23 SW_Push, SW24 SW_Push, SW25 SW_Push, SW26 SW_Push, SW27 SW_Push, SW28 SW_Push, SW29 SW_Push, SW3 SW_Push, SW30 SW_Push, SW31 SW_Push, SW32 SW_Push, SW33 SW_Push, SW34 SW_Push, SW35 SW_Push, SW36 SW_Push, SW37 SW_Push, SW38 SW_Push, SW39 SW_Push, SW4 SW_Push, SW40 SW_Push, SW41 SW_Push, SW42 SW_Push, SW43 SW_Push, SW44 SW_Push, SW45 SW_Push, SW46 SW_Push, SW47 SW_Push, SW48 SW_Push, SW49 SW_Push, SW5 SW_Push, SW50 SW_Push, SW51 SW_Push, SW52 SW_Push, SW53 SW_Push, SW54 SW_Push, SW55 SW_Push, SW56 SW_Push, SW57 SW_Push, SW58 SW_Push, SW59 SW_Push, SW6 SW_Push, SW60 SW_Push, SW61 SW_Push, SW62 SW_Push, SW63 SW_Push, SW64 SW_Push, SW65 SW_Push, SW66 SW_Push, SW67 SW_Push, SW68 SW_Push, SW69 SW_Push, SW7 SW_Push, SW70 SW_Push, SW71 SW_Push, SW72 SW_Push, SW73 SW_Push, SW74 SW_Push, SW75 SW_Push, SW76 SW_Push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

Commit message: ANSI-Alternativen: Backslash, Enter und linkes Shift
- SW106 Backslash 1.5u (ROW2/COL13): ohne LED, Schalter auf der Platine um
  270° gedreht – nur so kollidiert er nicht mit dem ISO-Enter-Stabilisator
- SW107 Enter 2.25u (ROW3/COL13) und SW108 Shift links 2.25u (ROW4/COL0)
  auf denselben Matrixpositionen wie ISO-Enter bzw. ISO-Shift
- ISO-Enter SW71 im Schaltplan um 180° gedreht: Pin 2 = COL13, Pin 1 = Diode
- Footprints mit dem Schaltplan verknüpft (Pfade fehlten seit kbplacer)
- kbplacer-Leiterbahnen entfernt: sie laufen durch die LED-Pads der
  kommenden Beleuchtung, das Routing wird ohnehin neu gemacht

DRC: nur erwartete NPTH-Überlappungen zwischen ISO- und ANSI-Footprints
(Stabi-/Befestigungslöcher) und der noch fehlende Platinenumriss.

Co-Authored-By: Claude Opus 5 (1M context) <noreply@anthropic.com>
Parts:
- added D106, D107, D108: D, Diode_SMD:D_SOD-123, symbol Device:D_Small
- added SW106: SW_Push, MX_Only:MXOnly-1.5U-NoLED, symbol Switch:SW_Push_45deg
- added SW107, SW108: SW_Push, MX_Only:MXOnly-2.25U-NoLED, symbol Switch:SW_Push_45deg
Connections:
- net COL0: now also SW108.1
- net COL13: now also SW71.2, SW106.2, SW107.1; no longer SW71.1
- net ROW2: now also D106.1 (K)
- net ROW3: now also D107.1 (K)
- net ROW4: now also D108.1 (K)
- net at D71.2 (A): now also SW71.1; no longer SW71.2
- new net: D106.2 (A), SW106.1
- new net: D108.2 (A), SW108.2
- new net: D107.2 (A), SW107.2
Other:
- note added: "ANSI alternatives - populate instead of the matching ISO keys SW106 Backslash 1.5u: no LED, switch rotated 270° on the PCB (clears the ISO Enter stabilizer) SW107 Enter 2.25u: same matrix position as ISO Enter SW71 (ROW3 / COL13) SW108 Left Shift 2.25u: same matrix position as ISO Left Shift SW75 (ROW4 / COL0) SW71 is drawn rotated 180°: pin 2 = COL13, pin 1 = diode (keeps its pads clear of SW106)"
- title: (none) -> convertible-keyboard-pcb
- moved on the sheet: SW71

Commit message: Einfarbige Hintergrundbeleuchtung (LEDs optional)
- Neues Symbol keyboard:SW_MX_LED: Einheit A Schalter (Pins wie
  SW_Push_45deg), Einheit B LED mit Pin 3 = Anode, Pin 4 = Kathode –
  passend zu den ai03-LED-Footprints (KiCads SW_Push_LED ist umgekehrt belegt)
- Alle Schalter außer ANSI-Backslash auf LED-Footprints umgestellt
- Blatt "Backlight": je Taste LED-Einheit + 1k-Vorwiderstand an +5V,
  Kathoden auf BL_K; AO3400A low-side als PWM-Treiber (BL_PWM)
- Caps-Lock- (SW58) und Num-Lock-LED (SW34) als Lock-Anzeige mit eigenem
  2N7002-Treiber (CAPS_LED, NUM_LED)
- LED-Kathode bei SW71, SW76, SW107 auf die andere Seite gelegt (FLIPPED),
  sonst zu nah an den Stabi-Löchern der ISO/ANSI-Alternativtaste;
  für ISO-Enter eigener Footprint lib/keyboard.pretty/MXOnly-ISO-FLIPPED
- Vorwiderstände auf B.Cu neben den Schaltern, bei den Alternativtasten
  in freie Bereiche verschoben

ERC meldet noch die unverbundenen Treiber-Eingänge und fehlende
Versorgungsquelle – beides kommt mit dem MCU-Blatt.

Co-Authored-By: Claude Opus 5 (1M context) <noreply@anthropic.com>
Parts:
- removed SW107, SW108: SW_Push, MX_Only:MXOnly-2.25U-NoLED, symbol Switch:SW_Push_45deg
- added SW107: SW_MX_LED, MX_Only:MXOnly-2.25U-FLIPPED, symbol keyboard:SW_MX_LED
- added SW108: SW_MX_LED, MX_Only:MXOnly-2.25U, symbol keyboard:SW_MX_LED
- SW1, SW10, SW101, SW102, SW103, SW105, SW11, SW12, SW13, SW14, SW15, SW16, SW17, SW18, SW19, SW2, SW20, SW21, SW22, SW23, SW24, SW25, SW26, SW27, SW28, SW29, SW3, SW31, SW32, SW33, SW34, SW35, SW36, SW37, SW39, SW4, SW40, SW41, SW42, SW43, SW44, SW45, SW46, SW47, SW48, SW49, SW5, SW50, SW51, SW52, SW53, SW54, SW55, SW56, SW59, SW6, SW60, SW61, SW62, SW63, SW64, SW65, SW66, SW67, SW68, SW69, SW7, SW70, SW72, SW73, SW74, SW77, SW78, SW79, SW8, SW80, SW81, SW82, SW83, SW84, SW85, SW86, SW88, SW89, SW9, SW90, SW91: value SW_Push -> SW_MX_LED; footprint MX_Only:MXOnly-1U-NoLED -> MX_Only:MXOnly-1U; symbol Switch:SW_Push_45deg -> keyboard:SW_MX_LED
- SW100, SW75, SW93, SW94, SW95, SW97, SW98, SW99: value SW_Push -> SW_MX_LED; footprint MX_Only:MXOnly-1.25U-NoLED -> MX_Only:MXOnly-1.25U; symbol Switch:SW_Push_45deg -> keyboard:SW_MX_LED
- SW104, SW30: value SW_Push -> SW_MX_LED; footprint MX_Only:MXOnly-2U-NoLED -> MX_Only:MXOnly-2U; symbol Switch:SW_Push_45deg -> keyboard:SW_MX_LED
- SW38: value SW_Push -> SW_MX_LED; footprint MX_Only:MXOnly-1.5U-NoLED -> MX_Only:MXOnly-1.5U; symbol Switch:SW_Push_45deg -> keyboard:SW_MX_LED
- SW57, SW92: value SW_Push -> SW_MX_LED; footprint MX_Only:MXOnly-2U-VerticalStabilizers-NoLED -> MX_Only:MXOnly-2U-VerticalStabilizers; symbol Switch:SW_Push_45deg -> keyboard:SW_MX_LED
- SW58: value SW_Push -> SW_MX_LED; footprint MX_Only:MXOnly-1.75U-NoLED -> MX_Only:MXOnly-1.75U; symbol Switch:SW_Push_45deg -> keyboard:SW_MX_LED
- SW71: value SW_Push -> SW_MX_LED; footprint MX_Only:MXOnly-ISO-NoLED -> keyboard:MXOnly-ISO-FLIPPED; symbol Switch:SW_Push_45deg -> keyboard:SW_MX_LED
- SW76: value SW_Push -> SW_MX_LED; footprint MX_Only:MXOnly-1U-NoLED -> MX_Only:MXOnly-1U-FLIPPED; symbol Switch:SW_Push_45deg -> keyboard:SW_MX_LED
- SW87: value SW_Push -> SW_MX_LED; footprint MX_Only:MXOnly-2.75U-NoLED -> MX_Only:MXOnly-2.75U; symbol Switch:SW_Push_45deg -> keyboard:SW_MX_LED
- SW96: value SW_Push -> SW_MX_LED; footprint MX_Only:MXOnly-6.25U-NoLED -> MX_Only:MXOnly-6.25U; symbol Switch:SW_Push_45deg -> keyboard:SW_MX_LED
Connections:
- net COL0: now also SW108.1
- net COL13: now also SW107.1
- net at D108.2 (A): now also SW108.2
- net at D107.2 (A): now also SW107.2
Other:
- added sheet Backlight (backlight.kicad_sch)

Commit message: MCU-Blatt: RP2040, USB-C, Stromversorgung; README und CLAUDE.md
- Blatt "MCU": RP2040 (QFN-56) mit W25Q16JVSS-Flash, 12-MHz-Quarz,
  AP2112K-3.3, USB-C (HRO TYPE-C-31-M-12, CC 5k1) mit USBLC6-2SC6,
  500-mA-Polyfuse, 27-Ω-Serienwiderständen, RESET- und BOOTSEL-Taster,
  SWD-Testpads, Entkopplung je Versorgungspin
- Alle 30 GPIOs belegt: GPIO0–20 COL0–20, GPIO21–26 ROW0–5,
  GPIO27 BL_PWM, GPIO28 CAPS_LED, GPIO29 NUM_LED
- Stabile UUIDs in den erzeugten Blättern, Beschriftungen aufgeräumt
- Neue Bauteile mit dem Schaltplan verknüpft, vorerst unplatziert unterhalb
  der Tasten

ERC: 0 Meldungen, Parität sauber. DRC: nur fehlender Umriss, die gewollten
ISO/ANSI-NPTH-Überlappungen und zwei Silkscreen-Hinweise.

Co-Authored-By: Claude Opus 5 (1M context) <noreply@anthropic.com>
Other:
- added sheet MCU (mcu.kicad_sch)
