File: convertible-keyboard-pcb.kicad_sch (KiCad schematic)
At the start: 216 parts, among them SW1 SW_MX_LED, SW10 SW_MX_LED, SW100 SW_MX_LED, SW101 SW_MX_LED, SW102 SW_MX_LED, SW103 SW_MX_LED, SW104 SW_MX_LED, SW105 SW_MX_LED, SW106 SW_Push, SW107 SW_MX_LED, SW108 SW_MX_LED, SW11 SW_MX_LED, SW12 SW_MX_LED, SW13 SW_MX_LED, SW14 SW_MX_LED, SW15 SW_MX_LED, SW16 SW_MX_LED, SW17 SW_MX_LED, SW18 SW_MX_LED, SW19 SW_MX_LED, SW2 SW_MX_LED, SW20 SW_MX_LED, SW21 SW_MX_LED, SW22 SW_MX_LED, SW23 SW_MX_LED, SW24 SW_MX_LED, SW25 SW_MX_LED, SW26 SW_MX_LED, SW27 SW_MX_LED, SW28 SW_MX_LED, SW29 SW_MX_LED, SW3 SW_MX_LED, SW30 SW_MX_LED, SW31 SW_MX_LED, SW32 SW_MX_LED, SW33 SW_MX_LED, SW34 SW_MX_LED, SW35 SW_MX_LED, SW36 SW_MX_LED, SW37 SW_MX_LED, SW38 SW_MX_LED, SW39 SW_MX_LED, SW4 SW_MX_LED, SW40 SW_MX_LED, SW41 SW_MX_LED, SW42 SW_MX_LED, SW43 SW_MX_LED, SW44 SW_MX_LED, SW45 SW_MX_LED, SW46 SW_MX_LED, SW47 SW_MX_LED, SW48 SW_MX_LED, SW49 SW_MX_LED, SW5 SW_MX_LED, SW50 SW_MX_LED, SW51 SW_MX_LED, SW52 SW_MX_LED, SW53 SW_MX_LED, SW54 SW_MX_LED, SW55 SW_MX_LED, SW56 SW_MX_LED, SW57 SW_MX_LED, SW58 SW_MX_LED, SW59 SW_MX_LED, SW6 SW_MX_LED, SW60 SW_MX_LED, SW61 SW_MX_LED, SW62 SW_MX_LED, SW63 SW_MX_LED, SW64 SW_MX_LED, SW65 SW_MX_LED, SW66 SW_MX_LED, SW67 SW_MX_LED, SW68 SW_MX_LED, SW69 SW_MX_LED, SW7 SW_MX_LED, SW70 SW_MX_LED, SW71 SW_MX_LED, SW72 SW_MX_LED, SW73 SW_MX_LED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

Commit message: Tasten-LEDs als Reverse-Mount-SMD (Standard), THT-Variante vorgehalten
- Schalter wieder mit 2-Pin-Symbol und ai03-NoLED-Footprints; jede Taste
  hat eine eigene LED LEDn (gleiche Nummer) auf der Rückseite unter dem
  LED-Fenster (Schaltermitte +5,08 mm) – Drähte und Netze unverändert
- LED: XINGLIGHT XL-3216UWC-FB, weiß, LCSC C3646935, maschinell bestückt
- Eigener Footprint LED_1206_ReverseMount_XL-3216 nach dem JLC/EasyEDA-
  Footprint (Pads 1,0 x 1,524 mm bei +-1,651, Aussparung 2,2 x 1,9 mm):
  Pad-Innenkante 0,2 mm von der Aussparung, Eckradius 0,5 mm zum Fräsen.
  KiCads generischer Reverse-Mount-Footprint passt nicht zu diesem Teil
  (Loch in Längsrichtung kleiner als die Linse)
- convertible-keyboard-pcb.kicad_dru: 0,2 mm Kantenabstand nur an den
  LED-Aussparungen, sonst weiter 0,5 mm
- tools/led_variant.py smd|tht: tauscht nur die LED-Footprints; THT-Pads
  als MX_LED_THT/_FLIPPED in lib/keyboard.pretty, Hin- und Rückweg getestet
- Entfernt: Symbol SW_MX_LED, sym-lib-table, MXOnly-ISO-FLIPPED
  (FLIPPED-Sonderfälle entfallen mit den NoLED-Schaltern)
- README (EN/DE), tools/README, CLAUDE.md aktualisiert

ERC 0, Parität sauber, DRC ohne Fehler (nur bekannte Warnungen).

Co-Authored-By: Claude Opus 5 (1M context) <noreply@anthropic.com>
Parts:
- SW1, SW10, SW101, SW102, SW103, SW105, SW11, SW12, SW13, SW14, SW15, SW16, SW17, SW18, SW19, SW2, SW20, SW21, SW22, SW23, SW24, SW25, SW26, SW27, SW28, SW29, SW3, SW31, SW32, SW33, SW34, SW35, SW36, SW37, SW39, SW4, SW40, SW41, SW42, SW43, SW44, SW45, SW46, SW47, SW48, SW49, SW5, SW50, SW51, SW52, SW53, SW54, SW55, SW56, SW59, SW6, SW60, SW61, SW62, SW63, SW64, SW65, SW66, SW67, SW68, SW69, SW7, SW70, SW72, SW73, SW74, SW77, SW78, SW79, SW8, SW80, SW81, SW82, SW83, SW84, SW85, SW86, SW88, SW89, SW9, SW90, SW91: value SW_MX_LED -> SW_Push; footprint MX_Only:MXOnly-1U -> MX_Only:MXOnly-1U-NoLED; symbol keyboard:SW_MX_LED -> Switch:SW_Push_45deg
- SW100, SW75, SW93, SW94, SW95, SW97, SW98, SW99: value SW_MX_LED -> SW_Push; footprint MX_Only:MXOnly-1.25U -> MX_Only:MXOnly-1.25U-NoLED; symbol keyboard:SW_MX_LED -> Switch:SW_Push_45deg
- SW104, SW30: value SW_MX_LED -> SW_Push; footprint MX_Only:MXOnly-2U -> MX_Only:MXOnly-2U-NoLED; symbol keyboard:SW_MX_LED -> Switch:SW_Push_45deg
- SW107: value SW_MX_LED -> SW_Push; footprint MX_Only:MXOnly-2.25U-FLIPPED -> MX_Only:MXOnly-2.25U-NoLED; symbol keyboard:SW_MX_LED -> Switch:SW_Push_45deg
- SW108: value SW_MX_LED -> SW_Push; footprint MX_Only:MXOnly-2.25U -> MX_Only:MXOnly-2.25U-NoLED; symbol keyboard:SW_MX_LED -> Switch:SW_Push_45deg
- SW38: value SW_MX_LED -> SW_Push; footprint MX_Only:MXOnly-1.5U -> MX_Only:MXOnly-1.5U-NoLED; symbol keyboard:SW_MX_LED -> Switch:SW_Push_45deg
- SW57, SW92: value SW_MX_LED -> SW_Push; footprint MX_Only:MXOnly-2U-VerticalStabilizers -> MX_Only:MXOnly-2U-VerticalStabilizers-NoLED; symbol keyboard:SW_MX_LED -> Switch:SW_Push_45deg
- SW58: value SW_MX_LED -> SW_Push; footprint MX_Only:MXOnly-1.75U -> MX_Only:MXOnly-1.75U-NoLED; symbol keyboard:SW_MX_LED -> Switch:SW_Push_45deg
- SW71: value SW_MX_LED -> SW_Push; footprint keyboard:MXOnly-ISO-FLIPPED -> MX_Only:MXOnly-ISO-NoLED; symbol keyboard:SW_MX_LED -> Switch:SW_Push_45deg
- SW76: value SW_MX_LED -> SW_Push; footprint MX_Only:MXOnly-1U-FLIPPED -> MX_Only:MXOnly-1U-NoLED; symbol keyboard:SW_MX_LED -> Switch:SW_Push_45deg
- SW87: value SW_MX_LED -> SW_Push; footprint MX_Only:MXOnly-2.75U -> MX_Only:MXOnly-2.75U-NoLED; symbol keyboard:SW_MX_LED -> Switch:SW_Push_45deg
- SW96: value SW_MX_LED -> SW_Push; footprint MX_Only:MXOnly-6.25U -> MX_Only:MXOnly-6.25U-NoLED; symbol keyboard:SW_MX_LED -> Switch:SW_Push_45deg

Commit message: Befestigungslöcher, LCSC-Nummern und Fertigungsdaten für JLCPCB
14 Befestigungslöcher (M2, NPTH, board_only) in die freien Flächen gesetzt;
endgültige Lage gemeinsam mit dem Gehäuse-Designer. Footprint dafür aus der
KiCad-Bibliothek ins Repo kopiert, damit es eigenständig bleibt.

LCSC/MPN/Manufacturer an allen 373 Symbolen und zusätzlich an den Footprints –
ohne die Felder am Footprint meldet die Schaltplan-Parität für jedes Bauteil ein
fehlendes Symbolfeld. Alle Nummern gegen Wert und Bauform geprüft.

Fertigungsdaten in docs/production/ mit zweisprachiger Anleitung: Gerber-ZIP
(ausdrücklich auf die 9 nötigen Lagen beschränkt, sonst landen Courtyard-, Fab-
und User-Lagen mit im Archiv), Bohrdatei mit PTH und NPTH gemeinsam, BOM und CPL
ohne die handgelöteten Schalter und ohne die DNP-Teile D122/J2/J3. Die
Y-Koordinaten der CPL bleiben negativ, passend zum Koordinatensystem der Gerber.

Dabei zwei Routing-Reste beseitigt: ein doppeltes RUN-Via, dessen Bohrung mit dem
Nachbarvia zusammenlief, und 13 deckungsgleiche Bahnsegmente. Die READMEs sagten
außerdem noch einseitige Bestückung – D126/D128 liegen auf F.Cu, der Auftrag ist
beidseitig.

Co-Authored-By: Claude Opus 5 (1M context) <noreply@anthropic.com>
Claude-Session: https://claude.ai/code/session_019Bb524k282LjrfvEdpjuYy
Parts:
- D1, D10, D100, D101, D102, D103, D104, D105, D106, D107, D108, D11, D12, D13, D14, D15, D16, D17, D18, D19, D2, D20, D21, D22, D23, D24, D25, D26, D27, D28, D29, D3, D30, D31, D32, D33, D34, D35, D36, D37, D38, D39, D4, D40, D41, D42, D43, D44, D45, D46, D47, D48, D49, D5, D50, D51, D52, D53, D54, D55, D56, D57, D58, D59, D6, D60, D61, D62, D63, D64, D65, D66, D67, D68, D69, D7, D70, D71, D72, D73, D74, D75, D76, D77, D78, D79, D8, D80, D81, D82, D83, D84, D85, D86, D87, D88, D89, D9, D90, D91, D92, D93, D94, D95, D96, D97, D98, D99: LCSC (none) -> C81598; MPN (none) -> 1N4148W; Manufacturer (none) -> CJ(Changjiang Elec)
