File: backlight.kicad_sch (KiCad schematic)
At the start: 223 parts, among them Q1 AO3400A, Q2 2N7002, Q3 2N7002, SW1 SW_MX_LED, SW10 SW_MX_LED, SW100 SW_MX_LED, SW101 SW_MX_LED, SW102 SW_MX_LED, SW103 SW_MX_LED, SW104 SW_MX_LED, SW105 SW_MX_LED, SW107 SW_MX_LED, SW108 SW_MX_LED, SW11 SW_MX_LED, SW12 SW_MX_LED, SW13 SW_MX_LED, SW14 SW_MX_LED, SW15 SW_MX_LED, SW16 SW_MX_LED, SW17 SW_MX_LED, SW18 SW_MX_LED, SW19 SW_MX_LED, SW2 SW_MX_LED, SW20 SW_MX_LED, SW21 SW_MX_LED, SW22 SW_MX_LED, SW23 SW_MX_LED, SW24 SW_MX_LED, SW25 SW_MX_LED, SW26 SW_MX_LED, SW27 SW_MX_LED, SW28 SW_MX_LED, SW29 SW_MX_LED, SW3 SW_MX_LED, SW30 SW_MX_LED, SW31 SW_MX_LED, SW32 SW_MX_LED, SW33 SW_MX_LED, SW34 SW_MX_LED, SW35 SW_MX_LED, SW36 SW_MX_LED, SW37 SW_MX_LED, SW38 SW_MX_LED, SW39 SW_MX_LED, SW4 SW_MX_LED, SW40 SW_MX_LED, SW41 SW_MX_LED, SW42 SW_MX_LED, SW43 SW_MX_LED, SW44 SW_MX_LED, SW45 SW_MX_LED, SW46 SW_MX_LED, SW47 SW_MX_LED, SW48 SW_MX_LED, SW49 SW_MX_LED, SW5 SW_MX_LED, SW50 SW_MX_LED, SW51 SW_MX_LED, SW52 SW_MX_LED, SW53 SW_MX_LED, SW54 SW_MX_LED, SW55 SW_MX_LED, SW56 SW_MX_LED, SW57 SW_MX_LED, SW58 SW_MX_LED, SW59 SW_MX_LED, SW6 SW_MX_LED, SW60 SW_MX_LED, SW61 SW_MX_LED, SW62 SW_MX_LED, SW63 SW_MX_LED, SW64 SW_MX_LED, SW65 SW_MX_LED, SW66 SW_MX_LED, SW67 SW_MX_LED, SW68 SW_MX_LED, SW69 SW_MX_LED, SW7 SW_MX_LED, SW70 SW_MX_LED, SW71 SW_MX_LED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

Commit message: Eigene Caps-/Num-Lock-Anzeige über dem Navigationsblock
- Caps- und Num-Taste gehören wieder zur normalen Beleuchtung (BL_K) –
  bei eingeschaltetem Licht war der Lock-Zustand in der Taste kaum erkennbar
- Je Anzeige 1k an +5V und zwei LEDs parallel zur Wahl: 3 mm THT
  (D121 Caps, D123 Num) oder 0805 SMD (D122, D124), Treiber Q2/Q3 wie bisher
- Platz im Spalt zwischen Druck/Rollen/Pause und Einfg/Pos1/BildAuf, also auf
  dem TKL-Teil: bleibt auch nach dem Abbrechen des Ziffernblocks erhalten
- tools/sync_pcb.py: feste Positionen über "absolute" in place_override.json
- README (EN/DE) und CLAUDE.md angepasst

ERC 0, Parität sauber.

Co-Authored-By: Claude Opus 5 (1M context) <noreply@anthropic.com>
Parts:
- added D121, D123: 3mm, LED_THT:LED_D3.0mm, symbol Device:LED_Small
- added D122, D124: 0805, LED_SMD:LED_0805_2012Metric, symbol Device:LED_Small
- added R127, R128: 1k, Resistor_SMD:R_0603_1608Metric, symbol Device:R_Small
Connections:
- net +5V: now also R127.1, R128.1
- net BL_K: now also SW34.4 (K), SW58.4 (K)
- net CAPS_K: now also D121.1 (K), D122.1 (K); no longer SW58.4 (K)
- net NUM_K: now also D123.1 (K), D124.1 (K); no longer SW34.4 (K)
- new net: D121.2 (A), D122.2 (A), R127.2
- new net: D123.2 (A), D124.2 (A), R128.2
Other:
- note added: "Backlight - every lit key has its own LED (unit B of the switch symbol) and series resistor. The through-hole LEDs are optional; resistors and drivers are always populated. LED pin 3 = anode, pin 4 = cathode. 1k gives about 2 mA per white LED at 5 V. Caps Lock and Num Lock have separate indicator LEDs above the navigation cluster (bottom right). SW106 (ANSI backslash) has no LED."
- note added: "Caps Lock"
- note added: "Lock indicators above the navigation cluster - populate either the 3 mm THT or the 0805 LED"
- note added: "Num Lock"
- note removed: "Backlight - every lit key has its own LED (unit B of the switch symbol) and series resistor. The through-hole LEDs are optional; resistors and drivers are always populated. LED pin 3 = anode, pin 4 = cathode. 1k gives about 2 mA per white LED at 5 V. Caps Lock (SW58) and Num Lock (SW34) LEDs are lock indicators with their own drivers. SW106 (ANSI backslash) has no LED."

Commit message: Lock-Anzeigen zusätzlich klassisch über dem Numpad (Standard)
- Zweites Paar Caps-/Num-Lock-Anzeigen rechts oben über dem Numpad:
  0805 bestückt (D126 Caps, D128 Num), 3-mm-THT vorgesehen (D125, D127, DNP)
- Paar über dem Navigationsblock bleibt für die TKL vorgesehen, alle LEDs DNP
- Jede Position mit eigenem 1k (R127–R130, bestückt), damit auch beide Paare
  gleichzeitig mit voller Helligkeit gehen; Treiber Q2/Q3 unverändert
- DNP wird in tools/sync_pcb.py auf die Footprints übertragen
- Generator: UUIDs zählen pro Blatt, Blatt-UUIDs hängen am Dateinamen –
  Ergänzungen auf einem Blatt verschieben die anderen nicht mehr
  (einmalige UUID-Änderung in allen erzeugten Blättern)
- README (EN/DE): beide Positionen, Wahl liegt beim Gehäuse-Designer

ERC 0, Parität sauber, DRC ohne neue Fehler.

Co-Authored-By: Claude Opus 5 (1M context) <noreply@anthropic.com>
Parts:
- added D125, D127: 3mm, LED_THT:LED_D3.0mm, symbol Device:LED_Small
- added D126, D128: 0805, LED_SMD:LED_0805_2012Metric, symbol Device:LED_Small
- added R129, R130: 1k, Resistor_SMD:R_0603_1608Metric, symbol Device:R_Small
- D121, D122, D123, D124: now not fitted
Connections:
- net +5V: now also R129.1, R130.1
- net CAPS_K: now also D125.1 (K), D126.1 (K)
- net NUM_K: now also D127.1 (K), D128.1 (K)
- new net: D125.2 (A), D126.2 (A), R129.2
- new net: D127.2 (A), D128.2 (A), R130.2
Other:
- note added: "Caps - nav (opt.)"
- note added: "Caps - numpad"
- note added: "Lock indicators - standard above the numpad (0805 populated), optional above the navigation cluster for the TKL (DNP). Every position takes a 3 mm THT or an 0805 LED; populate what the case needs."
- note added: "Num - nav (opt.)"
- note added: "Num - numpad"
- note removed: "Caps Lock"
- note removed: "Lock indicators above the navigation cluster - populate either the 3 mm THT or the 0805 LED"
- note removed: "Num Lock"
