File: backlight.kicad_sch (KiCad schematic)
At the start: 235 parts, among them Q1 AO3400A, Q2 2N7002, Q3 2N7002, SW1 SW_MX_LED, SW10 SW_MX_LED, SW100 SW_MX_LED, SW101 SW_MX_LED, SW102 SW_MX_LED, SW103 SW_MX_LED, SW104 SW_MX_LED, SW105 SW_MX_LED, SW107 SW_MX_LED, SW108 SW_MX_LED, SW11 SW_MX_LED, SW12 SW_MX_LED, SW13 SW_MX_LED, SW14 SW_MX_LED, SW15 SW_MX_LED, SW16 SW_MX_LED, SW17 SW_MX_LED, SW18 SW_MX_LED, SW19 SW_MX_LED, SW2 SW_MX_LED, SW20 SW_MX_LED, SW21 SW_MX_LED, SW22 SW_MX_LED, SW23 SW_MX_LED, SW24 SW_MX_LED, SW25 SW_MX_LED, SW26 SW_MX_LED, SW27 SW_MX_LED, SW28 SW_MX_LED, SW29 SW_MX_LED, SW3 SW_MX_LED, SW30 SW_MX_LED, SW31 SW_MX_LED, SW32 SW_MX_LED, SW33 SW_MX_LED, SW34 SW_MX_LED, SW35 SW_MX_LED, SW36 SW_MX_LED, SW37 SW_MX_LED, SW38 SW_MX_LED, SW39 SW_MX_LED, SW4 SW_MX_LED, SW40 SW_MX_LED, SW41 SW_MX_LED, SW42 SW_MX_LED, SW43 SW_MX_LED, SW44 SW_MX_LED, SW45 SW_MX_LED, SW46 SW_MX_LED, SW47 SW_MX_LED, SW48 SW_MX_LED, SW49 SW_MX_LED, SW5 SW_MX_LED, SW50 SW_MX_LED, SW51 SW_MX_LED, SW52 SW_MX_LED, SW53 SW_MX_LED, SW54 SW_MX_LED, SW55 SW_MX_LED, SW56 SW_MX_LED, SW57 SW_MX_LED, SW58 SW_MX_LED, SW59 SW_MX_LED, SW6 SW_MX_LED, SW60 SW_MX_LED, SW61 SW_MX_LED, SW62 SW_MX_LED, SW63 SW_MX_LED, SW64 SW_MX_LED, SW65 SW_MX_LED, SW66 SW_MX_LED, SW67 SW_MX_LED, SW68 SW_MX_LED, SW69 SW_MX_LED, SW7 SW_MX_LED, SW70 SW_MX_LED, SW71 SW_MX_LED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

Commit message: Blattgröße, Titelblöcke und Kommentare angepasst
Other:
- company: convertible-keyboard-pcb -> Philipp Weber
