File: backlight.kicad_sch (KiCad schematic)
At the start: 235 parts, among them Q1 AO3400A, Q2 2N7002, Q3 2N7002, SW1 SW_MX_LED, SW10 SW_MX_LED, SW100 SW_MX_LED, SW101 SW_MX_LED, SW102 SW_MX_LED, SW103 SW_MX_LED, SW104 SW_MX_LED, SW105 SW_MX_LED, SW107 SW_MX_LED, SW108 SW_MX_LED, SW11 SW_MX_LED, SW12 SW_MX_LED, SW13 SW_MX_LED, SW14 SW_MX_LED, SW15 SW_MX_LED, SW16 SW_MX_LED, SW17 SW_MX_LED, SW18 SW_MX_LED, SW19 SW_MX_LED, SW2 SW_MX_LED, SW20 SW_MX_LED, SW21 SW_MX_LED, SW22 SW_MX_LED, SW23 SW_MX_LED, SW24 SW_MX_LED, SW25 SW_MX_LED, SW26 SW_MX_LED, SW27 SW_MX_LED, SW28 SW_MX_LED, SW29 SW_MX_LED, SW3 SW_MX_LED, SW30 SW_MX_LED, SW31 SW_MX_LED, SW32 SW_MX_LED, SW33 SW_MX_LED, SW34 SW_MX_LED, SW35 SW_MX_LED, SW36 SW_MX_LED, SW37 SW_MX_LED, SW38 SW_MX_LED, SW39 SW_MX_LED, SW4 SW_MX_LED, SW40 SW_MX_LED, SW41 SW_MX_LED, SW42 SW_MX_LED, SW43 SW_MX_LED, SW44 SW_MX_LED, SW45 SW_MX_LED, SW46 SW_MX_LED, SW47 SW_MX_LED, SW48 SW_MX_LED, SW49 SW_MX_LED, SW5 SW_MX_LED, SW50 SW_MX_LED, SW51 SW_MX_LED, SW52 SW_MX_LED, SW53 SW_MX_LED, SW54 SW_MX_LED, SW55 SW_MX_LED, SW56 SW_MX_LED, SW57 SW_MX_LED, SW58 SW_MX_LED, SW59 SW_MX_LED, SW6 SW_MX_LED, SW60 SW_MX_LED, SW61 SW_MX_LED, SW62 SW_MX_LED, SW63 SW_MX_LED, SW64 SW_MX_LED, SW65 SW_MX_LED, SW66 SW_MX_LED, SW67 SW_MX_LED, SW68 SW_MX_LED, SW69 SW_MX_LED, SW7 SW_MX_LED, SW70 SW_MX_LED, SW71 SW_MX_LED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

Commit message: Lock-Anzeigen nur noch als 0805, TKL nur Caps Lock über BildAuf
- 3-mm-THT-Varianten entfernt (D121, D123, D125, D127)
- Über dem Numpad: D128 Num und D126 Caps mittig auf Höhe der F-Reihe,
  bestückt
- TKL: nur noch Caps Lock (D122, DNP) mittig über BildAuf in der Lücke
  zwischen F-Reihe und Zahlenreihe – Num Lock fällt mit dem Numpad ohnehin
  weg, daher Num-Anzeige D124 samt R128 entfernt
- Direkt in KiCad-Dateien geändert, nicht über tools/ – Generator-Stand
  endet mit 2eb5d4f (in tools/README und CLAUDE.md vermerkt)

ERC 0, Parität sauber, DRC ohne neue Meldungen.

Co-Authored-By: Claude Opus 5 (1M context) <noreply@anthropic.com>
Parts:
- removed D121, D123, D125, D127: 3mm, LED_THT:LED_D3.0mm, symbol Device:LED_Small
- removed D124: 0805, LED_SMD:LED_0805_2012Metric, symbol Device:LED_Small
- removed R128: 1k, Resistor_SMD:R_0603_1608Metric, symbol Device:R_Small
Other:
- note added: "Backlight - every lit key has its own LED (unit B of the switch symbol) and series resistor. The through-hole LEDs are optional; resistors and drivers are always populated. LED pin 3 = anode, pin 4 = cathode. 1k gives about 2 mA per white LED at 5 V. Caps Lock and Num Lock have separate 0805 indicator LEDs (bottom right). SW106 (ANSI backslash) has no LED."
- note added: "Caps - above PgUp (TKL, DNP)"
- note added: "Lock indicators (0805) - Num Lock and Caps Lock above the numpad, populated. For the TKL: Caps Lock above Page Up (DNP) - Num Lock goes with the numpad anyway."
- note removed: "Backlight - every lit key has its own LED (unit B of the switch symbol) and series resistor. The through-hole LEDs are optional; resistors and drivers are always populated. LED pin 3 = anode, pin 4 = cathode. 1k gives about 2 mA per white LED at 5 V. Caps Lock and Num Lock have separate indicator LEDs above the navigation cluster (bottom right). SW106 (ANSI backslash) has no LED."
- note removed: "Caps - nav (opt.)"
- note removed: "Lock indicators - standard above the numpad (0805 populated), optional above the navigation cluster for the TKL (DNP). Every position takes a 3 mm THT or an 0805 LED; populate what the case needs."
- note removed: "Num - nav (opt.)"
- moved on the sheet: D122, D126, D128, R127

Commit message: Tasten-LEDs als Reverse-Mount-SMD (Standard), THT-Variante vorgehalten
- Schalter wieder mit 2-Pin-Symbol und ai03-NoLED-Footprints; jede Taste
  hat eine eigene LED LEDn (gleiche Nummer) auf der Rückseite unter dem
  LED-Fenster (Schaltermitte +5,08 mm) – Drähte und Netze unverändert
- LED: XINGLIGHT XL-3216UWC-FB, weiß, LCSC C3646935, maschinell bestückt
- Eigener Footprint LED_1206_ReverseMount_XL-3216 nach dem JLC/EasyEDA-
  Footprint (Pads 1,0 x 1,524 mm bei +-1,651, Aussparung 2,2 x 1,9 mm):
  Pad-Innenkante 0,2 mm von der Aussparung, Eckradius 0,5 mm zum Fräsen.
  KiCads generischer Reverse-Mount-Footprint passt nicht zu diesem Teil
  (Loch in Längsrichtung kleiner als die Linse)
- convertible-keyboard-pcb.kicad_dru: 0,2 mm Kantenabstand nur an den
  LED-Aussparungen, sonst weiter 0,5 mm
- tools/led_variant.py smd|tht: tauscht nur die LED-Footprints; THT-Pads
  als MX_LED_THT/_FLIPPED in lib/keyboard.pretty, Hin- und Rückweg getestet
- Entfernt: Symbol SW_MX_LED, sym-lib-table, MXOnly-ISO-FLIPPED
  (FLIPPED-Sonderfälle entfallen mit den NoLED-Schaltern)
- README (EN/DE), tools/README, CLAUDE.md aktualisiert

ERC 0, Parität sauber, DRC ohne Fehler (nur bekannte Warnungen).

Co-Authored-By: Claude Opus 5 (1M context) <noreply@anthropic.com>
Parts:
- LED1: renamed from SW1; value SW_MX_LED -> XL-3216UWC-FB; footprint MX_Only:MXOnly-1U -> keyboard:LED_1206_ReverseMount_XL-3216; symbol keyboard:SW_MX_LED -> Device:LED_Small; LCSC (none) -> C3646935
- LED10: renamed from SW10; value SW_MX_LED -> XL-3216UWC-FB; footprint MX_Only:MXOnly-1U -> keyboard:LED_1206_ReverseMount_XL-3216; symbol keyboard:SW_MX_LED -> Device:LED_Small; LCSC (none) -> C3646935
- LED100: renamed from SW100; value SW_MX_LED -> XL-3216UWC-FB; footprint MX_Only:MXOnly-1.25U -> keyboard:LED_1206_ReverseMount_XL-3216; symbol keyboard:SW_MX_LED -> Device:LED_Small; LCSC (none) -> C3646935
- LED101: renamed from SW101; value SW_MX_LED -> XL-3216UWC-FB; footprint MX_Only:MXOnly-1U -> keyboard:LED_1206_ReverseMount_XL-3216; symbol keyboard:SW_MX_LED -> Device:LED_Small; LCSC (none) -> C3646935
- LED102: renamed from SW102; value SW_MX_LED -> XL-3216UWC-FB; footprint MX_Only:MXOnly-1U -> keyboard:LED_1206_ReverseMount_XL-3216; symbol keyboard:SW_MX_LED -> Device:LED_Small; LCSC (none) -> C3646935
- LED103: renamed from SW103; value SW_MX_LED -> XL-3216UWC-FB; footprint MX_Only:MXOnly-1U -> keyboard:LED_1206_ReverseMount_XL-3216; symbol keyboard:SW_MX_LED -> Device:LED_Small; LCSC (none) -> C3646935
- LED104: renamed from SW104; value SW_MX_LED -> XL-3216UWC-FB; footprint MX_Only:MXOnly-2U -> keyboard:LED_1206_ReverseMount_XL-3216; symbol keyboard:SW_MX_LED -> Device:LED_Small; LCSC (none) -> C3646935
- LED105: renamed from SW105; value SW_MX_LED -> XL-3216UWC-FB; footprint MX_Only:MXOnly-1U -> keyboard:LED_1206_ReverseMount_XL-3216; symbol keyboard:SW_MX_LED -> Device:LED_Small; LCSC (none) -> C3646935
- LED107: renamed from SW107; value SW_MX_LED -> XL-3216UWC-FB; footprint MX_Only:MXOnly-2.25U-FLIPPED -> keyboard:LED_1206_ReverseMount_XL-3216; symbol keyboard:SW_MX_LED -> Device:LED_Small; LCSC (none) -> C3646935
- LED108: renamed from SW108; value SW_MX_LED -> XL-3216UWC-FB; footprint MX_Only:MXOnly-2.25U -> keyboard:LED_1206_ReverseMount_XL-3216; symbol keyboard:SW_MX_LED -> Device:LED_Small; LCSC (none) -> C3646935
- LED11: renamed from SW11; value SW_MX_LED -> XL-3216UWC-FB; footprint MX_Only:MXOnly-1U -> keyboard:LED_1206_ReverseMount_XL-3216; symbol keyboard:SW_MX_LED -> Device:LED_Small; LCSC (none) -> C3646935
- LED12: renamed from SW12; value SW_MX_LED -> XL-3216UWC-FB; footprint MX_Only:MXOnly-1U -> keyboard:LED_1206_ReverseMount_XL-3216; symbol keyboard:SW_MX_LED -> Device:LED_Small; LCSC (none) -> C3646935
- LED13: renamed from SW13; value SW_MX_LED -> XL-3216UWC-FB; footprint MX_Only:MXOnly-1U -> keyboard:LED_1206_ReverseMount_XL-3216; symbol keyboard:SW_MX_LED -> Device:LED_Small; LCSC (none) -> C3646935
- LED14: renamed from SW14; value SW_MX_LED -> XL-3216UWC-FB; footprint MX_Only:MXOnly-1U -> keyboard:LED_1206_ReverseMount_XL-3216; symbol keyboard:SW_MX_LED -> Device:LED_Small; LCSC (none) -> C3646935
- LED15: renamed from SW15; value SW_MX_LED -> XL-3216UWC-FB; footprint MX_Only:MXOnly-1U -> keyboard:LED_1206_ReverseMount_XL-3216; symbol keyboard:SW_MX_LED -> Device:LED_Small; LCSC (none) -> C3646935
- LED16: renamed from SW16; value SW_MX_LED -> XL-3216UWC-FB; footprint MX_Only:MXOnly-1U -> keyboard:LED_1206_ReverseMount_XL-3216; symbol keyboard:SW_MX_LED -> Device:LED_Small; LCSC (none) -> C3646935
- LED17: renamed from SW17; value SW_MX_LED -> XL-3216UWC-FB; footprint MX_Only:MXOnly-1U -> keyboard:LED_1206_ReverseMount_XL-3216; symbol keyboard:SW_MX_LED -> Device:LED_Small; LCSC (none) -> C3646935
- LED18: renamed from SW18; value SW_MX_LED -> XL-3216UWC-FB; footprint MX_Only:MXOnly-1U -> keyboard:LED_1206_ReverseMount_XL-3216; symbol keyboard:SW_MX_LED -> Device:LED_Small; LCSC (none) -> C3646935
- LED19: renamed from SW19; value SW_MX_LED -> XL-3216UWC-FB; footprint MX_Only:MXOnly-1U -> keyboard:LED_1206_ReverseMount_XL-3216; symbol keyboard:SW_MX_LED -> Device:LED_Small; LCSC (none) -> C3646935
- LED2: renamed from SW2; value SW_MX_LED -> XL-3216UWC-FB; footprint MX_Only:MXOnly-1U -> keyboard:LED_1206_ReverseMount_XL-3216; symbol keyboard:SW_MX_LED -> Device:LED_Small; LCSC (none) -> C3646935
- LED20: renamed from SW20; value SW_MX_LED -> XL-3216UWC-FB; footprint MX_Only:MXOnly-1U -> keyboard:LED_1206_ReverseMount_XL-3216; symbol keyboard:SW_MX_LED -> Device:LED_Small; LCSC (none) -> C3646935
- LED21: renamed from SW21; value SW_MX_LED -> XL-3216UWC-FB; footprint MX_Only:MXOnly-1U -> keyboard:LED_1206_ReverseMount_XL-3216; symbol keyboard:SW_MX_LED -> Device:LED_Small; LCSC (none) -> C3646935
- LED22: renamed from SW22; value SW_MX_LED -> XL-3216UWC-FB; footprint MX_Only:MXOnly-1U -> keyboard:LED_1206_ReverseMount_XL-3216; symbol keyboard:SW_MX_LED -> Device:LED_Small; LCSC (none) -> C3646935
- LED23: renamed from SW23; value SW_MX_LED -> XL-3216UWC-FB; footprint MX_Only:MXOnly-1U -> keyboard:LED_1206_ReverseMount_XL-3216; symbol keyboard:SW_MX_LED -> Device:LED_Small; LCSC (none) -> C3646935
- LED24: renamed from SW24; value SW_MX_LED -> XL-3216UWC-FB; footprint MX_Only:MXOnly-1U -> keyboard:LED_1206_ReverseMount_XL-3216; symbol keyboard:SW_MX_LED -> Device:LED_Small; LCSC (none) -> C3646935
- LED25: renamed from SW25; value SW_MX_LED -> XL-3216UWC-FB; footprint MX_Only:MXOnly-1U -> keyboard:LED_1206_ReverseMount_XL-3216; symbol keyboard:SW_MX_LED -> Device:LED_Small; LCSC (none) -> C3646935
- LED26: renamed from SW26; value SW_MX_LED -> XL-3216UWC-FB; footprint MX_Only:MXOnly-1U -> keyboard:LED_1206_ReverseMount_XL-3216; symbol keyboard:SW_MX_LED -> Device:LED_Small; LCSC (none) -> C3646935
- LED27: renamed from SW27; value SW_MX_LED -> XL-3216UWC-FB; footprint MX_Only:MXOnly-1U -> keyboard:LED_1206_ReverseMount_XL-3216; symbol keyboard:SW_MX_LED -> Device:LED_Small; LCSC (none) -> C3646935
- LED28: renamed from SW28; value SW_MX_LED -> XL-3216UWC-FB; footprint MX_Only:MXOnly-1U -> keyboard:LED_1206_ReverseMount_XL-3216; symbol keyboard:SW_MX_LED -> Device:LED_Small; LCSC (none) -> C3646935
- LED29: renamed from SW29; value SW_MX_LED -> XL-3216UWC-FB; footprint MX_Only:MXOnly-1U -> keyboard:LED_1206_ReverseMount_XL-3216; symbol keyboard:SW_MX_LED -> Device:LED_Small; LCSC (none) -> C3646935
- LED3: renamed from SW3; value SW_MX_LED -> XL-3216UWC-FB; footprint MX_Only:MXOnly-1U -> keyboard:LED_1206_ReverseMount_XL-3216; symbol keyboard:SW_MX_LED -> Device:LED_Small; LCSC (none) -> C3646935
- LED30: renamed from SW30; value SW_MX_LED -> XL-3216UWC-FB; footprint MX_Only:MXOnly-2U -> keyboard:LED_1206_ReverseMount_XL-3216; symbol keyboard:SW_MX_LED -> Device:LED_Small; LCSC (none) -> C3646935
- LED31: renamed from SW31; value SW_MX_LED -> XL-3216UWC-FB; footprint MX_Only:MXOnly-1U -> keyboard:LED_1206_ReverseMount_XL-3216; symbol keyboard:SW_MX_LED -> Device:LED_Small; LCSC (none) -> C3646935
- LED32: renamed from SW32; value SW_MX_LED -> XL-3216UWC-FB; footprint MX_Only:MXOnly-1U -> keyboard:LED_1206_ReverseMount_XL-3216; symbol keyboard:SW_MX_LED -> Device:LED_Small; LCSC (none) -> C3646935
- LED33: renamed from SW33; value SW_MX_LED -> XL-3216UWC-FB; footprint MX_Only:MXOnly-1U -> keyboard:LED_1206_ReverseMount_XL-3216; symbol keyboard:SW_MX_LED -> Device:LED_Small; LCSC (none) -> C3646935
- LED34: renamed from SW34; value SW_MX_LED -> XL-3216UWC-FB; footprint MX_Only:MXOnly-1U -> keyboard:LED_1206_ReverseMount_XL-3216; symbol keyboard:SW_MX_LED -> Device:LED_Small; LCSC (none) -> C3646935
- LED35: renamed from SW35; value SW_MX_LED -> XL-3216UWC-FB; footprint MX_Only:MXOnly-1U -> keyboard:LED_1206_ReverseMount_XL-3216; symbol keyboard:SW_MX_LED -> Device:LED_Small; LCSC (none) -> C3646935
- LED36: renamed from SW36; value SW_MX_LED -> XL-3216UWC-FB; footprint MX_Only:MXOnly-1U -> keyboard:LED_1206_ReverseMount_XL-3216; symbol keyboard:SW_MX_LED -> Device:LED_Small; LCSC (none) -> C3646935
- LED37: renamed from SW37; value SW_MX_LED -> XL-3216UWC-FB; footprint MX_Only:MXOnly-1U -> keyboard:LED_1206_ReverseMount_XL-3216; symbol keyboard:SW_MX_LED -> Device:LED_Small; LCSC (none) -> C3646935
- LED38: renamed from SW38; value SW_MX_LED -> XL-3216UWC-FB; footprint MX_Only:MXOnly-1.5U -> keyboard:LED_1206_ReverseMount_XL-3216; symbol keyboard:SW_MX_LED -> Device:LED_Small; LCSC (none) -> C3646935
- LED39: renamed from SW39; value SW_MX_LED -> XL-3216UWC-FB; footprint MX_Only:MXOnly-1U -> keyboard:LED_1206_ReverseMount_XL-3216; symbol keyboard:SW_MX_LED -> Device:LED_Small; LCSC (none) -> C3646935
- LED4: renamed from SW4; value SW_MX_LED -> XL-3216UWC-FB; footprint MX_Only:MXOnly-1U -> keyboard:LED_1206_ReverseMount_XL-3216; symbol keyboard:SW_MX_LED -> Device:LED_Small; LCSC (none) -> C3646935
- LED40: renamed from SW40; value SW_MX_LED -> XL-3216UWC-FB; footprint MX_Only:MXOnly-1U -> keyboard:LED_1206_ReverseMount_XL-3216; symbol keyboard:SW_MX_LED -> Device:LED_Small; LCSC (none) -> C3646935
- LED41: renamed from SW41; value SW_MX_LED -> XL-3216UWC-FB; footprint MX_Only:MXOnly-1U -> keyboard:LED_1206_ReverseMount_XL-3216; symbol keyboard:SW_MX_LED -> Device:LED_Small; LCSC (none) -> C3646935
- LED42: renamed from SW42; value SW_MX_LED -> XL-3216UWC-FB; footprint MX_Only:MXOnly-1U -> keyboard:LED_1206_ReverseMount_XL-3216; symbol keyboard:SW_MX_LED -> Device:LED_Small; LCSC (none) -> C3646935
- LED43: renamed from SW43; value SW_MX_LED -> XL-3216UWC-FB; footprint MX_Only:MXOnly-1U -> keyboard:LED_1206_ReverseMount_XL-3216; symbol keyboard:SW_MX_LED -> Device:LED_Small; LCSC (none) -> C3646935
- LED44: renamed from SW44; value SW_MX_LED -> XL-3216UWC-FB; footprint MX_Only:MXOnly-1U -> keyboard:LED_1206_ReverseMount_XL-3216; symbol keyboard:SW_MX_LED -> Device:LED_Small; LCSC (none) -> C3646935
- LED45: renamed from SW45; value SW_MX_LED -> XL-3216UWC-FB; footprint MX_Only:MXOnly-1U -> keyboard:LED_1206_ReverseMount_XL-3216; symbol keyboard:SW_MX_LED -> Device:LED_Small; LCSC (none) -> C3646935
- LED46: renamed from SW46; value SW_MX_LED -> XL-3216UWC-FB; footprint MX_Only:MXOnly-1U -> keyboard:LED_1206_ReverseMount_XL-3216; symbol keyboard:SW_MX_LED -> Device:LED_Small; LCSC (none) -> C3646935
- LED47: renamed from SW47; value SW_MX_LED -> XL-3216UWC-FB; footprint MX_Only:MXOnly-1U -> keyboard:LED_1206_ReverseMount_XL-3216; symbol keyboard:SW_MX_LED -> Device:LED_Small; LCSC (none) -> C3646935
- LED48: renamed from SW48; value SW_MX_LED -> XL-3216UWC-FB; footprint MX_Only:MXOnly-1U -> keyboard:LED_1206_ReverseMount_XL-3216; symbol keyboard:SW_MX_LED -> Device:LED_Small; LCSC (none) -> C3646935
- LED49: renamed from SW49; value SW_MX_LED -> XL-3216UWC-FB; footprint MX_Only:MXOnly-1U -> keyboard:LED_1206_ReverseMount_XL-3216; symbol keyboard:SW_MX_LED -> Device:LED_Small; LCSC (none) -> C3646935
- LED5: renamed from SW5; value SW_MX_LED -> XL-3216UWC-FB; footprint MX_Only:MXOnly-1U -> keyboard:LED_1206_ReverseMount_XL-3216; symbol keyboard:SW_MX_LED -> Device:LED_Small; LCSC (none) -> C3646935
- LED50: renamed from SW50; value SW_MX_LED -> XL-3216UWC-FB; footprint MX_Only:MXOnly-1U -> keyboard:LED_1206_ReverseMount_XL-3216; symbol keyboard:SW_MX_LED -> Device:LED_Small; LCSC (none) -> C3646935
- LED51: renamed from SW51; value SW_MX_LED -> XL-3216UWC-FB; footprint MX_Only:MXOnly-1U -> keyboard:LED_1206_ReverseMount_XL-3216; symbol keyboard:SW_MX_LED -> Device:LED_Small; LCSC (none) -> C3646935
- LED52: renamed from SW52; value SW_MX_LED -> XL-3216UWC-FB; footprint MX_Only:MXOnly-1U -> keyboard:LED_1206_ReverseMount_XL-3216; symbol keyboard:SW_MX_LED -> Device:LED_Small; LCSC (none) -> C3646935
- LED53: renamed from SW53; value SW_MX_LED -> XL-3216UWC-FB; footprint MX_Only:MXOnly-1U -> keyboard:LED_1206_ReverseMount_XL-3216; symbol keyboard:SW_MX_LED -> Device:LED_Small; LCSC (none) -> C3646935
- LED54: renamed from SW54; value SW_MX_LED -> XL-3216UWC-FB; footprint MX_Only:MXOnly-1U -> keyboard:LED_1206_ReverseMount_XL-3216; symbol keyboard:SW_MX_LED -> Device:LED_Small; LCSC (none) -> C3646935
- LED55: renamed from SW55; value SW_MX_LED -> XL-3216UWC-FB; footprint MX_Only:MXOnly-1U -> keyboard:LED_1206_ReverseMount_XL-3216; symbol keyboard:SW_MX_LED -> Device:LED_Small; LCSC (none) -> C3646935
- LED56: renamed from SW56; value SW_MX_LED -> XL-3216UWC-FB; footprint MX_Only:MXOnly-1U -> keyboard:LED_1206_ReverseMount_XL-3216; symbol keyboard:SW_MX_LED -> Device:LED_Small; LCSC (none) -> C3646935
- LED57: renamed from SW57; value SW_MX_LED -> XL-3216UWC-FB; footprint MX_Only:MXOnly-2U-VerticalStabilizers -> keyboard:LED_1206_ReverseMount_XL-3216; symbol keyboard:SW_MX_LED -> Device:LED_Small; LCSC (none) -> C3646935
- LED58: renamed from SW58; value SW_MX_LED -> XL-3216UWC-FB; footprint MX_Only:MXOnly-1.75U -> keyboard:LED_1206_ReverseMount_XL-3216; symbol keyboard:SW_MX_LED -> Device:LED_Small; LCSC (none) -> C3646935
- LED59: renamed from SW59; value SW_MX_LED -> XL-3216UWC-FB; footprint MX_Only:MXOnly-1U -> keyboard:LED_1206_ReverseMount_XL-3216; symbol keyboard:SW_MX_LED -> Device:LED_Small; LCSC (none) -> C3646935
- LED6: renamed from SW6; value SW_MX_LED -> XL-3216UWC-FB; footprint MX_Only:MXOnly-1U -> keyboard:LED_1206_ReverseMount_XL-3216; symbol keyboard:SW_MX_LED -> Device:LED_Small; LCSC (none) -> C3646935
- LED60: renamed from SW60; value SW_MX_LED -> XL-3216UWC-FB; footprint MX_Only:MXOnly-1U -> keyboard:LED_1206_ReverseMount_XL-3216; symbol keyboard:SW_MX_LED -> Device:LED_Small; LCSC (none) -> C3646935
- LED61: renamed from SW61; value SW_MX_LED -> XL-3216UWC-FB; footprint MX_Only:MXOnly-1U -> keyboard:LED_1206_ReverseMount_XL-3216; symbol keyboard:SW_MX_LED -> Device:LED_Small; LCSC (none) -> C3646935
- LED62: renamed from SW62; value SW_MX_LED -> XL-3216UWC-FB; footprint MX_Only:MXOnly-1U -> keyboard:LED_1206_ReverseMount_XL-3216; symbol keyboard:SW_MX_LED -> Device:LED_Small; LCSC (none) -> C3646935
- LED63: renamed from SW63; value SW_MX_LED -> XL-3216UWC-FB; footprint MX_Only:MXOnly-1U -> keyboard:LED_1206_ReverseMount_XL-3216; symbol keyboard:SW_MX_LED -> Device:LED_Small; LCSC (none) -> C3646935
- LED64: renamed from SW64; value SW_MX_LED -> XL-3216UWC-FB; footprint MX_Only:MXOnly-1U -> keyboard:LED_1206_ReverseMount_XL-3216; symbol keyboard:SW_MX_LED -> Device:LED_Small; LCSC (none) -> C3646935
- LED65: renamed from SW65; value SW_MX_LED -> XL-3216UWC-FB; footprint MX_Only:MXOnly-1U -> keyboard:LED_1206_ReverseMount_XL-3216; symbol keyboard:SW_MX_LED -> Device:LED_Small; LCSC (none) -> C3646935
- LED66: renamed from SW66; value SW_MX_LED -> XL-3216UWC-FB; footprint MX_Only:MXOnly-1U -> keyboard:LED_1206_ReverseMount_XL-3216; symbol keyboard:SW_MX_LED -> Device:LED_Small; LCSC (none) -> C3646935
- LED67: renamed from SW67; value SW_MX_LED -> XL-3216UWC-FB; footprint MX_Only:MXOnly-1U -> keyboard:LED_1206_ReverseMount_XL-3216; symbol keyboard:SW_MX_LED -> Device:LED_Small; LCSC (none) -> C3646935
- LED68: renamed from SW68; value SW_MX_LED -> XL-3216UWC-FB; footprint MX_Only:MXOnly-1U -> keyboard:LED_1206_ReverseMount_XL-3216; symbol keyboard:SW_MX_LED -> Device:LED_Small; LCSC (none) -> C3646935
- LED69: renamed from SW69; value SW_MX_LED -> XL-3216UWC-FB; footprint MX_Only:MXOnly-1U -> keyboard:LED_1206_ReverseMount_XL-3216; symbol keyboard:SW_MX_LED -> Device:LED_Small; LCSC (none) -> C3646935
- LED7: renamed from SW7; value SW_MX_LED -> XL-3216UWC-FB; footprint MX_Only:MXOnly-1U -> keyboard:LED_1206_ReverseMount_XL-3216; symbol keyboard:SW_MX_LED -> Device:LED_Small; LCSC (none) -> C3646935
- LED70: renamed from SW70; value SW_MX_LED -> XL-3216UWC-FB; footprint MX_Only:MXOnly-1U -> keyboard:LED_1206_ReverseMount_XL-3216; symbol keyboard:SW_MX_LED -> Device:LED_Small; LCSC (none) -> C3646935
- LED71: renamed from SW71; value SW_MX_LED -> XL-3216UWC-FB; footprint keyboard:MXOnly-ISO-FLIPPED -> keyboard:LED_1206_ReverseMount_XL-3216; symbol keyboard:SW_MX_LED -> Device:LED_Small; LCSC (none) -> C3646935
- LED72: renamed from SW72; value SW_MX_LED -> XL-3216UWC-FB; footprint MX_Only:MXOnly-1U -> keyboard:LED_1206_ReverseMount_XL-3216; symbol keyboard:SW_MX_LED -> Device:LED_Small; LCSC (none) -> C3646935
- LED73: renamed from SW73; value SW_MX_LED -> XL-3216UWC-FB; footprint MX_Only:MXOnly-1U -> keyboard:LED_1206_ReverseMount_XL-3216; symbol keyboard:SW_MX_LED -> Device:LED_Small; LCSC (none) -> C3646935
- LED74: renamed from SW74; value SW_MX_LED -> XL-3216UWC-FB; footprint MX_Only:MXOnly-1U -> keyboard:LED_1206_ReverseMount_XL-3216; symbol keyboard:SW_MX_LED -> Device:LED_Small; LCSC (none) -> C3646935
- LED75: renamed from SW75; value SW_MX_LED -> XL-3216UWC-FB; footprint MX_Only:MXOnly-1.25U -> keyboard:LED_1206_ReverseMount_XL-3216; symbol keyboard:SW_MX_LED -> Device:LED_Small; LCSC (none) -> C3646935
- LED76: renamed from SW76; value SW_MX_LED -> XL-3216UWC-FB; footprint MX_Only:MXOnly-1U-FLIPPED -> keyboard:LED_1206_ReverseMount_XL-3216; symbol keyboard:SW_MX_LED -> Device:LED_Small; LCSC (none) -> C3646935
- LED77: renamed from SW77; value SW_MX_LED -> XL-3216UWC-FB; footprint MX_Only:MXOnly-1U -> keyboard:LED_1206_ReverseMount_XL-3216; symbol keyboard:SW_MX_LED -> Device:LED_Small; LCSC (none) -> C3646935
- LED78: renamed from SW78; value SW_MX_LED -> XL-3216UWC-FB; footprint MX_Only:MXOnly-1U -> keyboard:LED_1206_ReverseMount_XL-3216; symbol keyboard:SW_MX_LED -> Device:LED_Small; LCSC (none) -> C3646935
- LED79: renamed from SW79; value SW_MX_LED -> XL-3216UWC-FB; footprint MX_Only:MXOnly-1U -> keyboard:LED_1206_ReverseMount_XL-3216; symbol keyboard:SW_MX_LED -> Device:LED_Small; LCSC (none) -> C3646935
- LED8: renamed from SW8; value SW_MX_LED -> XL-3216UWC-FB; footprint MX_Only:MXOnly-1U -> keyboard:LED_1206_ReverseMount_XL-3216; symbol keyboard:SW_MX_LED -> Device:LED_Small; LCSC (none) -> C3646935
- LED80: renamed from SW80; value SW_MX_LED -> XL-3216UWC-FB; footprint MX_Only:MXOnly-1U -> keyboard:LED_1206_ReverseMount_XL-3216; symbol keyboard:SW_MX_LED -> Device:LED_Small; LCSC (none) -> C3646935
- LED81: renamed from SW81; value SW_MX_LED -> XL-3216UWC-FB; footprint MX_Only:MXOnly-1U -> keyboard:LED_1206_ReverseMount_XL-3216; symbol keyboard:SW_MX_LED -> Device:LED_Small; LCSC (none) -> C3646935
- LED82: renamed from SW82; value SW_MX_LED -> XL-3216UWC-FB; footprint MX_Only:MXOnly-1U -> keyboard:LED_1206_ReverseMount_XL-3216; symbol keyboard:SW_MX_LED -> Device:LED_Small; LCSC (none) -> C3646935
- LED83: renamed from SW83; value SW_MX_LED -> XL-3216UWC-FB; footprint MX_Only:MXOnly-1U -> keyboard:LED_1206_ReverseMount_XL-3216; symbol keyboard:SW_MX_LED -> Device:LED_Small; LCSC (none) -> C3646935
- LED84: renamed from SW84; value SW_MX_LED -> XL-3216UWC-FB; footprint MX_Only:MXOnly-1U -> keyboard:LED_1206_ReverseMount_XL-3216; symbol keyboard:SW_MX_LED -> Device:LED_Small; LCSC (none) -> C3646935
- LED85: renamed from SW85; value SW_MX_LED -> XL-3216UWC-FB; footprint MX_Only:MXOnly-1U -> keyboard:LED_1206_ReverseMount_XL-3216; symbol keyboard:SW_MX_LED -> Device:LED_Small; LCSC (none) -> C3646935
- LED86: renamed from SW86; value SW_MX_LED -> XL-3216UWC-FB; footprint MX_Only:MXOnly-1U -> keyboard:LED_1206_ReverseMount_XL-3216; symbol keyboard:SW_MX_LED -> Device:LED_Small; LCSC (none) -> C3646935
- LED87: renamed from SW87; value SW_MX_LED -> XL-3216UWC-FB; footprint MX_Only:MXOnly-2.75U -> keyboard:LED_1206_ReverseMount_XL-3216; symbol keyboard:SW_MX_LED -> Device:LED_Small; LCSC (none) -> C3646935
- LED88: renamed from SW88; value SW_MX_LED -> XL-3216UWC-FB; footprint MX_Only:MXOnly-1U -> keyboard:LED_1206_ReverseMount_XL-3216; symbol keyboard:SW_MX_LED -> Device:LED_Small; LCSC (none) -> C3646935
- LED89: renamed from SW89; value SW_MX_LED -> XL-3216UWC-FB; footprint MX_Only:MXOnly-1U -> keyboard:LED_1206_ReverseMount_XL-3216; symbol keyboard:SW_MX_LED -> Device:LED_Small; LCSC (none) -> C3646935
- LED9: renamed from SW9; value SW_MX_LED -> XL-3216UWC-FB; footprint MX_Only:MXOnly-1U -> keyboard:LED_1206_ReverseMount_XL-3216; symbol keyboard:SW_MX_LED -> Device:LED_Small; LCSC (none) -> C3646935
- LED90: renamed from SW90; value SW_MX_LED -> XL-3216UWC-FB; footprint MX_Only:MXOnly-1U -> keyboard:LED_1206_ReverseMount_XL-3216; symbol keyboard:SW_MX_LED -> Device:LED_Small; LCSC (none) -> C3646935
- LED91: renamed from SW91; value SW_MX_LED -> XL-3216UWC-FB; footprint MX_Only:MXOnly-1U -> keyboard:LED_1206_ReverseMount_XL-3216; symbol keyboard:SW_MX_LED -> Device:LED_Small; LCSC (none) -> C3646935
- LED92: renamed from SW92; value SW_MX_LED -> XL-3216UWC-FB; footprint MX_Only:MXOnly-2U-VerticalStabilizers -> keyboard:LED_1206_ReverseMount_XL-3216; symbol keyboard:SW_MX_LED -> Device:LED_Small; LCSC (none) -> C3646935
- LED93: renamed from SW93; value SW_MX_LED -> XL-3216UWC-FB; footprint MX_Only:MXOnly-1.25U -> keyboard:LED_1206_ReverseMount_XL-3216; symbol keyboard:SW_MX_LED -> Device:LED_Small; LCSC (none) -> C3646935
- LED94: renamed from SW94; value SW_MX_LED -> XL-3216UWC-FB; footprint MX_Only:MXOnly-1.25U -> keyboard:LED_1206_ReverseMount_XL-3216; symbol keyboard:SW_MX_LED -> Device:LED_Small; LCSC (none) -> C3646935
- LED95: renamed from SW95; value SW_MX_LED -> XL-3216UWC-FB; footprint MX_Only:MXOnly-1.25U -> keyboard:LED_1206_ReverseMount_XL-3216; symbol keyboard:SW_MX_LED -> Device:LED_Small; LCSC (none) -> C3646935
- LED96: renamed from SW96; value SW_MX_LED -> XL-3216UWC-FB; footprint MX_Only:MXOnly-6.25U -> keyboard:LED_1206_ReverseMount_XL-3216; symbol keyboard:SW_MX_LED -> Device:LED_Small; LCSC (none) -> C3646935
- LED97: renamed from SW97; value SW_MX_LED -> XL-3216UWC-FB; footprint MX_Only:MXOnly-1.25U -> keyboard:LED_1206_ReverseMount_XL-3216; symbol keyboard:SW_MX_LED -> Device:LED_Small; LCSC (none) -> C3646935
- LED98: renamed from SW98; value SW_MX_LED -> XL-3216UWC-FB; footprint MX_Only:MXOnly-1.25U -> keyboard:LED_1206_ReverseMount_XL-3216; symbol keyboard:SW_MX_LED -> Device:LED_Small; LCSC (none) -> C3646935
- LED99: renamed from SW99; value SW_MX_LED -> XL-3216UWC-FB; footprint MX_Only:MXOnly-1.25U -> keyboard:LED_1206_ReverseMount_XL-3216; symbol keyboard:SW_MX_LED -> Device:LED_Small; LCSC (none) -> C3646935
Connections:
- net BL_K: now also LED1.1 (K), LED10.1 (K), LED100.1 (K), LED101.1 (K), LED102.1 (K), LED103.1 (K), LED104.1 (K), LED105.1 (K), LED107.1 (K), LED108.1 (K), LED11.1 (K), LED12.1 (K), LED13.1 (K), LED14.1 (K), LED15.1 (K), LED16.1 (K), LED17.1 (K), LED18.1 (K), LED19.1 (K), LED2.1 (K), LED20.1 (K), LED21.1 (K), LED22.1 (K), LED23.1 (K), LED24.1 (K), LED25.1 (K), LED26.1 (K), LED27.1 (K), LED28.1 (K), LED29.1 (K), LED3.1 (K), LED30.1 (K), LED31.1 (K), LED32.1 (K), LED33.1 (K), LED34.1 (K), LED35.1 (K), LED36.1 (K), LED37.1 (K), LED38.1 (K)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; no longer LED1.4 (K), LED10.4 (K), LED100.4 (K), LED101.4 (K), LED102.4 (K), LED103.4 (K), LED104.4 (K), LED105.4 (K), LED107.4 (K), LED108.4 (K), LED11.4 (K), LED12.4 (K), LED13.4 (K), LED14.4 (K), LED15.4 (K), LED16.4 (K), LED17.4 (K), LED18.4 (K), LED19.4 (K), LED2.4 (K), LED20.4 (K), LED21.4 (K), LED22.4 (K), LED23.4 (K), LED24.4 (K), LED25.4 (K), LED26.4 (K), LED27.4 (K), LED28.4 (K), LED29.4 (K), LED3.4 (K), LED30.4 (K), LED31.4 (K), LED32.4 (K), LED33.4 (K), LED34.4 (K), LED35.4 (K), LED36.4 (K), LED37.4 (K), LED38.4 (K)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
- net at R48.2: now also LED48.2 (A); no longer LED48.3 (A)
- net at R12.2: now also LED12.2 (A); no longer LED12.3 (A)
- net at R32.2: now also LED32.2 (A); no longer LED32.3 (A)
- net at R15.2: now also LED15.2 (A); no longer LED15.3 (A)
- net at R67.2: now also LED67.2 (A); no longer LED67.3 (A)
- net at R46.2: now also LED46.2 (A); no longer LED46.3 (A)
- net at R61.2: now also LED61.2 (A); no longer LED61.3 (A)
- net at R22.2: now also LED22.2 (A); no longer LED22.3 (A)
- net at R47.2: now also LED47.2 (A); no longer LED47.3 (A)
- net at R75.2: now also LED75.2 (A); no longer LED75.3 (A)
- net at R13.2: now also LED13.2 (A); no longer LED13.3 (A)
- net at R2.2: now also LED2.2 (A); no longer LED2.3 (A)
- net at R77.2: now also LED77.2 (A); no longer LED77.3 (A)
- net at R68.2: now also LED68.2 (A); no longer LED68.3 (A)
- net at R90.2: now also LED90.2 (A); no longer LED90.3 (A)
- net at R43.2: now also LED43.2 (A); no longer LED43.3 (A)
- net at R42.2: now also LED42.2 (A); no longer LED42.3 (A)
- net at R60.2: now also LED60.2 (A); no longer LED60.3 (A)
- net at R58.2: now also LED58.2 (A); no longer LED58.3 (A)
- net at R99.2: now also LED99.2 (A); no longer LED99.3 (A)
- net at R100.2: now also LED100.2 (A); no longer LED100.3 (A)
- net at R92.2: now also LED92.2 (A); no longer LED92.3 (A)
- net at R53.2: now also LED53.2 (A); no longer LED53.3 (A)
- net at R85.2: now also LED85.2 (A); no longer LED85.3 (A)
- net at R59.2: now also LED59.2 (A); no longer LED59.3 (A)
- net at R98.2: now also LED98.2 (A); no longer LED98.3 (A)
- net at R95.2: now also LED95.2 (A); no longer LED95.3 (A)
- net at R10.2: now also LED10.2 (A); no longer LED10.3 (A)
- net at R66.2: now also LED66.2 (A); no longer LED66.3 (A)
- net at R50.2: now also LED50.2 (A); no longer LED50.3 (A)
- net at R6.2: now also LED6.2 (A); no longer LED6.3 (A)
- net at R102.2: now also LED102.2 (A); no longer LED102.3 (A)
- net at R27.2: now also LED27.2 (A); no longer LED27.3 (A)
- net at R64.2: now also LED64.2 (A); no longer LED64.3 (A)
- net at R1.2: now also LED1.2 (A); no longer LED1.3 (A)
- net at R63.2: now also LED63.2 (A); no longer LED63.3 (A)
- net at R57.2: now also LED57.2 (A); no longer LED57.3 (A)
- net at R69.2: now also LED69.2 (A); no longer LED69.3 (A)
- net at R104.2: now also LED104.2 (A); no longer LED104.3 (A)
- net at R19.2: now also LED19.2 (A); no longer LED19.3 (A)
- net at R71.2: now also LED71.2 (A); no longer LED71.3 (A)
- net at R26.2: now also LED26.2 (A); no longer LED26.3 (A)
- net at R28.2: now also LED28.2 (A); no longer LED28.3 (A)
- net at R101.2: now also LED101.2 (A); no longer LED101.3 (A)
- net at R107.2: now also LED107.2 (A); no longer LED107.3 (A)
- net at R62.2: now also LED62.2 (A); no longer LED62.3 (A)
- net at R5.2: now also LED5.2 (A); no longer LED5.3 (A)
- net at R55.2: now also LED55.2 (A); no longer LED55.3 (A)
- net at R76.2: now also LED76.2 (A); no longer LED76.3 (A)
- net at R73.2: now also LED73.2 (A); no longer LED73.3 (A)
- net at R41.2: now also LED41.2 (A); no longer LED41.3 (A)
- net at R11.2: now also LED11.2 (A); no longer LED11.3 (A)
- net at R35.2: now also LED35.2 (A); no longer LED35.3 (A)
- net at R105.2: now also LED105.2 (A); no longer LED105.3 (A)
- net at R89.2: now also LED89.2 (A); no longer LED89.3 (A)
- net at R25.2: now also LED25.2 (A); no longer LED25.3 (A)
- net at R38.2: now also LED38.2 (A); no longer LED38.3 (A)
- net at R8.2: now also LED8.2 (A); no longer LED8.3 (A)
- net at R36.2: now also LED36.2 (A); no longer LED36.3 (A)
- net at R18.2: now also LED18.2 (A); no longer LED18.3 (A)
- net at R54.2: now also LED54.2 (A); no longer LED54.3 (A)
- net at R108.2: now also LED108.2 (A); no longer LED108.3 (A)
- net at R44.2: now also LED44.2 (A); no longer LED44.3 (A)
- net at R51.2: now also LED51.2 (A); no longer LED51.3 (A)
- net at R96.2: now also LED96.2 (A); no longer LED96.3 (A)
- net at R88.2: now also LED88.2 (A); no longer LED88.3 (A)
- net at R31.2: now also LED31.2 (A); no longer LED31.3 (A)
- net at R86.2: now also LED86.2 (A); no longer LED86.3 (A)
- net at R9.2: now also LED9.2 (A); no longer LED9.3 (A)
- net at R79.2: now also LED79.2 (A); no longer LED79.3 (A)
- net at R80.2: now also LED80.2 (A); no longer LED80.3 (A)
- net at R37.2: now also LED37.2 (A); no longer LED37.3 (A)
- net at R56.2: now also LED56.2 (A); no longer LED56.3 (A)
- net at R24.2: now also LED24.2 (A); no longer LED24.3 (A)
- net at R72.2: now also LED72.2 (A); no longer LED72.3 (A)
- net at R14.2: now also LED14.2 (A); no longer LED14.3 (A)
- net at R84.2: now also LED84.2 (A); no longer LED84.3 (A)
- net at R33.2: now also LED33.2 (A); no longer LED33.3 (A)
- net at R93.2: now also LED93.2 (A); no longer LED93.3 (A)
- net at R94.2: now also LED94.2 (A); no longer LED94.3 (A)
- net at R52.2: now also LED52.2 (A); no longer LED52.3 (A)
- net at R83.2: now also LED83.2 (A); no longer LED83.3 (A)
- net at R4.2: now also LED4.2 (A); no longer LED4.3 (A)
- net at R82.2: now also LED82.2 (A); no longer LED82.3 (A)
- net at R39.2: now also LED39.2 (A); no longer LED39.3 (A)
- net at R87.2: now also LED87.2 (A); no longer LED87.3 (A)
- net at R78.2: now also LED78.2 (A); no longer LED78.3 (A)
- net at R45.2: now also LED45.2 (A); no longer LED45.3 (A)
- net at R65.2: now also LED65.2 (A); no longer LED65.3 (A)
- net at R29.2: now also LED29.2 (A); no longer LED29.3 (A)
- net at R3.2: now also LED3.2 (A); no longer LED3.3 (A)
- net at R16.2: now also LED16.2 (A); no longer LED16.3 (A)
- net at R97.2: now also LED97.2 (A); no longer LED97.3 (A)
- net at R74.2: now also LED74.2 (A); no longer LED74.3 (A)
- net at R103.2: now also LED103.2 (A); no longer LED103.3 (A)
- net at R34.2: now also LED34.2 (A); no longer LED34.3 (A)
- net at R20.2: now also LED20.2 (A); no longer LED20.3 (A)
- net at R91.2: now also LED91.2 (A); no longer LED91.3 (A)
- net at R49.2: now also LED49.2 (A); no longer LED49.3 (A)
- net at R23.2: now also LED23.2 (A); no longer LED23.3 (A)
- net at R40.2: now also LED40.2 (A); no longer LED40.3 (A)
- net at R7.2: now also LED7.2 (A); no longer LED7.3 (A)
- net at R81.2: now also LED81.2 (A); no longer LED81.3 (A)
- net at R17.2: now also LED17.2 (A); no longer LED17.3 (A)
- net at R21.2: now also LED21.2 (A); no longer LED21.3 (A)
- net at R30.2: now also LED30.2 (A); no longer LED30.3 (A)
- net at R70.2: now also LED70.2 (A); no longer LED70.3 (A)
Other:
- note added: "Backlight - every lit key has its own reverse-mount 1206 LED (LEDn, same number as the switch) and 1k series resistor. Standard: XINGLIGHT XL-3216UWC-FB, white (LCSC C3646935), on the back of the PCB, shining through the board into the switch's LED window. THT variant: same schematic, only the LED footprint changes (lib/keyboard.pretty MX_LED_THT, _FLIPPED at LED71/76/107). 1k gives about 1.6 mA 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"
- note removed: "Backlight - every lit key has its own LED (unit B of the switch symbol) and series resistor. The through-hole LEDs are optional; resistors and drivers are always populated. LED pin 3 = anode, pin 4 = cathode. 1k gives about 2 mA per white LED at 5 V. Caps Lock and Num Lock have separate 0805 indicator LEDs (bottom right). SW106 (ANSI backslash) has no LED."

Commit message: Platinenumriss und Sollbruchstelle, Alternativ-LEDs in der Stückliste
- Umriss: Tastenfeld + 1,3 mm rundum (Ecken r = 1 mm). Die 1,3 mm sind
  nötig, weil die Stabi-Löcher von Leertaste, Num 0 und Num+ über das reine
  Tastenfeld hinausragen. USB-C J1 sitzt bündig mit der Oberkante
- Sollbruchstelle: 2 mm breiter Schlitz bei x = 378,6 mit vier
  Mouse-Bite-Stegen (Footprint Breakaway_Tab_MouseBite, BRK1–BRK4). Jeder
  Steg hat einen lochfreien Kanal für bis zu drei Bahnen pro Lage:
  BRK1 COL17–COL20/CAPS_K/NUM_K, BRK2 ROW1/ROW2/+5V,
  BRK3 ROW3/ROW4/BL_K, BRK4 ROW5
- Tasten-LEDs mit Stücklistenfeldern Manufacturer, MPN und
  LCSC Alternatives (geprüft: C401114 MEIHUA MHT151WDT,
  C2827252 TUOZHAN P2-1206WYCS2-0.9T-F); Standard bleibt XL-3216UWC-FB.
  tools/led_variant.py pflegt die Felder mit
- README (EN/DE) und CLAUDE.md aktualisiert

ERC 0, Parität sauber, DRC ohne Fehler.

Co-Authored-By: Claude Opus 5 (1M context) <noreply@anthropic.com>
Parts:
- LED1, LED10, LED100, LED101, LED102, LED103, LED104, LED105, LED107, LED108, LED11, LED12, LED13, LED14, LED15, LED16, LED17, LED18, LED19, LED2, LED20, LED21, LED22, LED23, LED24, LED25, LED26, LED27, LED28, LED29, LED3, LED30, LED31, LED32, LED33, LED34, LED35, LED36, LED37, LED38, LED39, LED4, LED40, LED41, LED42, LED43, LED44, LED45, LED46, LED47, LED48, LED49, LED5, LED50, LED51, LED52, LED53, LED54, LED55, LED56, LED57, LED58, LED59, LED6, LED60, LED61, LED62, LED63, LED64, LED65, LED66, LED67, LED68, LED69, LED7, LED70, LED71, LED72, LED73, LED74, LED75, LED76, LED77, LED78, LED79, LED8, LED80, LED81, LED82, LED83, LED84, LED85, LED86, LED87, LED88, LED89, LED9, LED90, LED91, LED92, LED93, LED94, LED95, LED96, LED97, LED98, LED99: LCSC Alternatives (none) -> C401114 MEIHUA MHT151WDT; C2827252 TUOZHAN P2-1206WYCS2-0.9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; MPN (none) -> XL-3216UWC-FB; Manufacturer (none) -> XINGLIGHT

Commit message: Befestigungslöcher, LCSC-Nummern und Fertigungsdaten für JLCPCB
14 Befestigungslöcher (M2, NPTH, board_only) in die freien Flächen gesetzt;
endgültige Lage gemeinsam mit dem Gehäuse-Designer. Footprint dafür aus der
KiCad-Bibliothek ins Repo kopiert, damit es eigenständig bleibt.

LCSC/MPN/Manufacturer an allen 373 Symbolen und zusätzlich an den Footprints –
ohne die Felder am Footprint meldet die Schaltplan-Parität für jedes Bauteil ein
fehlendes Symbolfeld. Alle Nummern gegen Wert und Bauform geprüft.

Fertigungsdaten in docs/production/ mit zweisprachiger Anleitung: Gerber-ZIP
(ausdrücklich auf die 9 nötigen Lagen beschränkt, sonst landen Courtyard-, Fab-
und User-Lagen mit im Archiv), Bohrdatei mit PTH und NPTH gemeinsam, BOM und CPL
ohne die handgelöteten Schalter und ohne die DNP-Teile D122/J2/J3. Die
Y-Koordinaten der CPL bleiben negativ, passend zum Koordinatensystem der Gerber.

Dabei zwei Routing-Reste beseitigt: ein doppeltes RUN-Via, dessen Bohrung mit dem
Nachbarvia zusammenlief, und 13 deckungsgleiche Bahnsegmente. Die READMEs sagten
außerdem noch einseitige Bestückung – D126/D128 liegen auf F.Cu, der Auftrag ist
beidseitig.

Co-Authored-By: Claude Opus 5 (1M context) <noreply@anthropic.com>
Claude-Session: https://claude.ai/code/session_019Bb524k282LjrfvEdpjuYy
Parts:
- D122, D126, D128: LCSC (none) -> C34499; MPN (none) -> KT-0805W; Manufacturer (none) -> Hubei KENTO Elec
- Q1: LCSC (none) -> C20917; MPN (none) -> AO3400A; Manufacturer (none) -> Alpha & Omega
- Q2, Q3: LCSC (none) -> C8545; MPN (none) -> 2N7002; Manufacturer (none) -> CJ(Changjiang Elec)
- R1, R10, R100, R101, R102, R103, R104, R105, R107, R108, R11, R12, R127, R129, R13, R130, R14, R15, R16, R17, R18, R19, R2, R20, R21, R22, R23, R24, R25, R26, R27, R28, R29, R3, R30, R31, R32, R33, R34, R35, R36, R37, R38, R39, R4, R40, R41, R42, R43, R44, R45, R46, R47, R48, R49, R5, R50, R51, R52, R53, R54, R55, R56, R57, R58, R59, R6, R60, R61, R62, R63, R64, R65, R66, R67, R68, R69, R7, R70, R71, R72, R73, R74, R75, R76, R77, R78, R79, R8, R80, R81, R82, R83, R84, R85, R86, R87, R88, R89, R9, R90, R91, R92, R93, R94, R95, R96, R97, R98, R99: LCSC (none) -> C21190; MPN (none) -> 0603WAF1001T5E; Manufacturer (none) -> UNIROYAL ELEC
- R121, R123, R125: LCSC (none) -> C22775; MPN (none) -> 0603WAF1000T5E; Manufacturer (none) -> UNIROYAL ELEC
- R122, R124, R126: LCSC (none) -> C25803; MPN (none) -> 0603WAF1003T5E; Manufacturer (none) -> UNIROYAL ELEC
